File: examples/layout_reuse/layout/sub/sub.kicad_pcb (KiCad board)
At the start: 2 copper layers, 3 parts

Commit message: Restore Atopile Local 0.2 on pinned 0.15.9 sources
Import the publicly distributed atopile 0.15.9 PyPI source release as the
compiler/UI baseline, retaining upstream main as its historical parent.
PyPI source SHA256: 681cc1e123646dd133de31b631aedaf4eaac88682613b4f82d1da4b3ef8b4e8e.

Revive the local VS Code extension with a separate identity and launcher,
isolated state, bundled visualization assets, and provider settings. Bridge
the existing Atopile tool harness to a natively signed-in Codex app-server
for ChatGPT-plan use, retaining direct API providers as explicit options.
Include local part import, layout tools, packaging/runtime setup and tests.

Preserve upstream licensing, restored GitHub metadata and source notices.
Exclude local environments, generated webview bundles and personal QA paths.
Parts:
- R1, R2, R3: value 1kΩ -> 1kΩ ±1%
Changed lines of the file:
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@@
 			(usegerberadvancedattributes yes)
 			(creategerberjobfile yes)
-			(dashed_line_dash_ratio 12.000000)
-			(dashed_line_gap_ratio 3.000000)
+			(dashed_line_dash_ratio 12)
+			(dashed_line_gap_ratio 3)
 			(svgprecision 4)
 			(plotframeref no)
@@
 			(hpglpennumber 1)
 			(hpglpenspeed 20)
-			(hpglpendiameter 15.000000)
+			(hpglpendiameter 15)
 			(pdf_front_fp_property_popups yes)
 			(pdf_back_fp_property_popups yes)
@@
 			)
 		)
-		(property "Value" "1kΩ"
+		(property "Value" "1kΩ ±1%"
 			(at 0 4 90)
 			(layer "F.Fab")
@@
 			)
 		)
-		(property "resistance" "1±1.0%kΩ"
+		(property "resistance" "1kΩ ±1%"
 			(at 0 0 90)
 			(layer "User.9")
@@
 			)
 			(layer "F.SilkS")
+			(layers "F.SilkS")
+			(locked no)
 		)
 		(fp_line
@@
 			)
 			(layer "F.SilkS")
+			(layers "F.SilkS")
+			(locked no)
 		)
 		(fp_line
@@
 			)
 			(layer "F.SilkS")
+			(layers "F.SilkS")
+			(locked no)
 		)
 		(fp_line
@@
 			)
 			(layer "F.SilkS")
+			(layers "F.SilkS")
+			(locked no)
 		)
 		(fp_line
@@
 			)
 			(layer "F.SilkS")
+			(layers "F.SilkS")
+			(locked no)
 		)
 		(fp_line
@@
 			)
 			(layer "F.SilkS")
+			(layers "F.SilkS")
+			(locked no)
 		)
 		(fp_circle
@@
 				(type solid)
 			)
-			(fill no)
 			(layer "F.Fab")
-		)
-		(fp_text user "${REFERENCE}"
-			(at 0 0 90)
-			(layer "F.Fab")
-			(effects
-				(font
-					(size 1 1)
-					(thickness 0.15)
-				)
-			)
+			(locked no)
 		)
 		(pad "1" smd rect
 			(at -0.43 0 90)
 			(size 0.57 0.54)
-			(layers "F.Cu" "F.Mask" "F.Paste")
+			(layers "F.Cu" "F.Paste" "F.Mask")
 			(net 2 "unnamed[0]-2")
 		)
@@
 			(at 0.43 0 90)
 			(size 0.57 0.54)
-			(layers "F.Cu" "F.Mask" "F.Paste")
+			(layers "F.Cu" "F.Paste" "F.Mask")
 			(net 1 "unnamed[1]")
 		)
@@
 			)
 		)
-		(property "Value" "1kΩ"
+		(property "Value" "1kΩ ±1%"
 			(at 0 4 90)
 			(layer "F.Fab")
@@
 			)
 		)
-		(property "resistance" "1±1.0%kΩ"
+		(property "resistance" "1kΩ ±1%"
 			(at 0 0 90)
 			(layer "User.9")
@@
 			)
 			(layer "F.SilkS")
+			(layers "F.SilkS")
+			(locked no)
 		)
 		(fp_line
@@
 			)
 			(layer "F.SilkS")
+			(layers "F.SilkS")
+			(locked no)
 		)
 		(fp_line
@@
 			)
 			(layer "F.SilkS")
+			(layers "F.SilkS")
+			(locked no)
 		)
 		(fp_line
@@
 			)
 			(layer "F.SilkS")
+			(layers "F.SilkS")
+			(locked no)
 		)
 		(fp_line
@@
 			)
 			(layer "F.SilkS")
+			(layers "F.SilkS")
+			(locked no)
 		)
 		(fp_line
@@
 			)
 			(layer "F.SilkS")
+			(layers "F.SilkS")
+			(locked no)
 		)
 		(fp_circle
@@
 				(type solid)
 			)
-			(fill no)
 			(layer "F.Fab")
-		)
-		(fp_text user "${REFERENCE}"
-			(at 0 0 90)
-			(layer "F.Fab")
-			(effects
-				(font
-					(size 1 1)
-					(thickness 0.15)
-				)
-			)
+			(locked no)
 		)
 		(pad "1" smd rect
 			(at -0.43 0 90)
 			(size 0.57 0.54)
-			(layers "F.Cu" "F.Mask" "F.Paste")
+			(layers "F.Cu" "F.Paste" "F.Mask")
 			(net 3 "unnamed[0]-1")
 		)
@@
 			(at 0.43 0 90)
 			(size 0.57 0.54)
-			(layers "F.Cu" "F.Mask" "F.Paste")
+			(layers "F.Cu" "F.Paste" "F.Mask")
 			(net 2 "unnamed[0]-2")
 		)
@@
 			)
 		)
-		(property "Value" "1kΩ"
+		(property "Value" "1kΩ ±1%"
 			(at 0 4 90)
 			(layer "F.Fab")
@@
 			)
 		)
-		(property "resistance" "1±1.0%kΩ"
+		(property "resistance" "1kΩ ±1%"
 			(at 0 0 90)
 			(layer "User.9")
@@
 			)
 			(layer "F.SilkS")
+			(layers "F.SilkS")
+			(locked no)
 		)
 		(fp_line
@@
 			)
 			(layer "F.SilkS")
+			(layers "F.SilkS")
+			(locked no)
 		)
 		(fp_line
@@
 			)
 			(layer "F.SilkS")
+			(layers "F.SilkS")
+			(locked no)
 		)
 		(fp_line
@@
 			)
 			(layer "F.SilkS")
+			(layers "F.SilkS")
+			(locked no)
 		)
 		(fp_line
@@
 			)
 			(layer "F.SilkS")
+			(layers "F.SilkS")
+			(locked no)
 		)
 		(fp_line
@@
 			)
 			(layer "F.SilkS")
+			(layers "F.SilkS")
+			(locked no)
 		)
 		(fp_circle
@@
 				(type solid)
 			)
-			(fill no)
 			(layer "F.Fab")
-		)
-		(fp_text user "${REFERENCE}"
-			(at 0 0 90)
-			(layer "F.Fab")
-			(effects
-				(font
-					(size 1 1)
-					(thickness 0.15)
-				)
-			)
+			(locked no)
 		)
 		(pad "1" smd rect
 			(at -0.43 0 90)
 			(size 0.57 0.54)
-			(layers "F.Cu" "F.Mask" "F.Paste")
+			(layers "F.Cu" "F.Paste" "F.Mask")
 			(net 4 "unnamed[0]")
 		)
@@
 			(at 0.43 0 90)
 			(size 0.57 0.54)
-			(layers "F.Cu" "F.Mask" "F.Paste")
+			(layers "F.Cu" "F.Paste" "F.Mask")
 			(net 3 "unnamed[0]-1")
 		)
