File: projects/chrysler-scanner/current/ChryslerScanner_V240_SD.kicad_sch (KiCad schematic)
At the start: 0 parts

Commit message: Finish scanner routing and add hierarchical system schematics
Other:
- sheet OBD line protection renamed OBD connector + protection
- removed sheet OBD connector
- sheet 5 V / 3.3 V supplies ports: added +12V, +3.3V, +5V, GND; removed none
- sheet 7.5 V supply ports: added +12V, +7.5V, GND; removed none
- sheet CCD interface ports: added +3.3V, +5V, GND, J1962-11, J1962-3, RX1, TBEN, TX1; removed none
- sheet ESP32 + RF ports: added +3.3V, ACT_LED, EN, GND, IO0, LOG_BUTTON, MCU_SD_CS, MCU_SD_MOSI, MCU_SD_SCK, N_R25_1, PCI_RX, PCI_TX, PWR_LED, RX0, RX1, RX2, RX_LED, SCL, SDA, SD_DETECT, SD_MISO, TX1, TX2, TX_LED, V_BA, V_BT, V_PR; removed none
- sheet I/O expander + I2C ports: added +3.3V, +5V, GND, RX15_EN, RX7_BIAS_EN, RX7_EN, SCL, SDA, TBEN, TX12_EN, TX14_EN, TX6_EN, TX9_EN, VBB_TO_TX12, VBB_TO_TX14, VBB_TO_TX6, VBB_TO_TX9, VPP_TO_TX12, VPP_TO_TX14, VPP_TO_TX6, VPP_TO_TX9; removed none
- sheet Integrated SD logger ports: added +3.3V, +5V, GND, LOG_BUTTON, MCU_SD_CS, MCU_SD_MOSI, MCU_SD_SCK, SD_DETECT, SD_MISO; removed none
- sheet OBD connector + protection ports: added GND, J1962-11, J1962-12, J1962-14, J1962-15, J1962-16, J1962-2, J1962-3, J1962-6, J1962-7, J1962-9, N_J1_5, N_Q1B_3; removed none
- sheet PCI / J1850 ports: added +12V, +3.3V, +5V, +7.5V, GND, J1962-2, N_Q1B_3, PCI_RX, PCI_TX; removed none
- sheet SCI RX7 / RX15 ports: added +3.3V, +5V, GND, J1962-15, J1962-7, RX15_EN, RX2, RX7_BIAS, RX7_EN; removed none
- sheet SCI TX12 VBB / VPP drivers ports: added GND, J1962-12, VBB, VBB_TO_TX12, VPP, VPP_TO_TX12; removed none
- sheet SCI TX14 / TX9 ports: added +3.3V, +5V, GND, J1962-14, J1962-9, TX14_EN, TX2, TX9_EN; removed none
- sheet SCI TX14 VBB / VPP drivers ports: added GND, J1962-14, VBB, VBB_TO_TX14, VPP, VPP_TO_TX14; removed none
- sheet SCI TX6 / TX12 + RX bias ports: added +3.3V, +5V, GND, J1962-12, J1962-6, RX7_BIAS, RX7_BIAS_EN, TX12_EN, TX2, TX6_EN; removed none
- sheet SCI TX6 VBB / VPP drivers ports: added GND, J1962-6, VBB, VBB_TO_TX6, VPP, VPP_TO_TX6; removed none
- sheet SCI TX9 VBB / VPP drivers ports: added GND, J1962-9, VBB, VBB_TO_TX9, VPP, VPP_TO_TX9; removed none
- sheet Status LED drivers ports: added +3.3V, +5V, ACT_LED, GND, PWR_LED, RX_LED, TX_LED; removed none
- sheet USB + reset / boot ports: added +3.3V, +5V, EN, GND, IO0, N_R25_1, RX0; removed none
- sheet VBB supply ports: added GND, VBB, VPP; removed none
- sheet VPP boost supply ports: added +12V, +5V, GND, VPP; removed none
- sheet Vehicle power input ports: added +12V, GND, J1962-16, N_J1_5; removed none
- sheet Voltage monitoring ports: added GND, J1962-16, VBB, VPP, V_BA, V_BT, V_PR; removed none
- note added: "Named signal stubs connect the same net across blocks. Click a block to open its circuit. J1 and input protection share one sheet."
- note added: "SYSTEM BLOCK DIAGRAM / HIERARCHICAL SIGNALS"
- note removed: "1 parts / page 22"
- note removed: "10 parts / page 10"
- note removed: "10 parts / page 11"
- note removed: "11 parts / page 7"
- note removed: "12 parts / page 18"
- note removed: "12 parts / page 3"
- note removed: "12 parts / page 5"
- note removed: "15 parts / page 12"
- note removed: "16 parts / page 17"
- note removed: "16 parts / page 21"
- note removed: "17 parts / page 9"
- note removed: "18 added parts / page 23"
- note removed: "19 parts / page 20"
- note removed: "25 parts / page 2"
- note removed: "259 components | 154 nets | 23 native KiCad pages | integrated SD revision"
- note removed: "4 parts / page 8"
- note removed: "7 parts / page 19"
- note removed: "9 parts / page 13"
- note removed: "9 parts / page 14"
- note removed: "9 parts / page 15"
- note removed: "9 parts / page 16"
- note removed: "9 parts / page 4"
- note removed: "9 parts / page 6"
- note removed: "ChryslerScanner V240-USB-C-OBD-SD-A"
- note removed: "Open a sheet to inspect symbols and wires. Matching signal names connect across sheets."
- note removed: "Passive pin types: connectivity checked, independent electrical review still required."
- note removed: "Preserves USB-C, ATTEND OBD-II and scanner functions. SD hardware added; firmware remains deferred."
- note removed: "U3 / U4 / U8 pin 5 is connected to GND; corrected to match the PCB and source netlist."
- title: ChryslerScanner V240-USB-C-OBD | circuit overview -> ChryslerScanner V240 - system hierarchy

Commit message: Restore functional system diagram layout with hierarchical signals
Other:
- note added: "ADC"
- note added: "AW9523B | bus enables and programming control"
- note added: "BUS INTERFACES"
- note added: "Battery / GND"
- note added: "Bus data"
- note added: "CONTROL & SENSING"
- note added: "ChryslerScanner V240 | integrated microSD | 259 components | 154 connected nets"
- note added: "Double-click a block to open its circuit. Native hierarchical pins and named stubs carry the exact design nets."
- note added: "Enables / bias"
- note added: "HOST & LOGGING"
- note added: "I2C"
- note added: "J1 and input protection share one sheet. Solid arrows show data flow; native named stubs define electrical connectivity."
- note added: "J2 USB-C | CP2102 bridge | reset / boot"
- note added: "J4 microSD | SD_3V3 | LOG / STOP"
- note added: "POWER GENERATION & SCI PROGRAMMING"
- note added: "Protected supply"
- note added: "SCI stages"
- note added: "SPI / detect"
- note added: "SYSTEM BLOCK DIAGRAM"
- note added: "Separate VBB / VPP rails feed the SCI programming stages; enables come from AW9523B."
- note added: "Solid arrows: data and user interface paths. Dashed arrows: power or control relationships."
- note added: "Status"
- note added: "UART / reset"
- note added: "VEHICLE CONNECTION"
- note removed: "Named signal stubs connect the same net across blocks. Click a block to open its circuit. J1 and input protection share one sheet."
- note removed: "SYSTEM BLOCK DIAGRAM / HIERARCHICAL SIGNALS"
- title: ChryslerScanner V240 - system hierarchy -> ChryslerScanner V240 - system block diagram

Commit message: Use native ground symbols and document companion app feasibility
Other:
- sheet 5 V / 3.3 V supplies ports: added none; removed GND
- sheet 7.5 V supply ports: added none; removed GND
- sheet CCD interface ports: added none; removed GND
- sheet ESP32 + RF ports: added none; removed GND
- sheet I/O expander + I2C ports: added none; removed GND
- sheet Integrated SD logger ports: added none; removed GND
- sheet OBD connector + protection ports: added none; removed GND
- sheet PCI / J1850 ports: added none; removed GND
- sheet SCI RX7 / RX15 ports: added none; removed GND
- sheet SCI TX12 VBB / VPP drivers ports: added none; removed GND
- sheet SCI TX14 / TX9 ports: added none; removed GND
- sheet SCI TX14 VBB / VPP drivers ports: added none; removed GND
- sheet SCI TX6 / TX12 + RX bias ports: added none; removed GND
- sheet SCI TX6 VBB / VPP drivers ports: added none; removed GND
- sheet SCI TX9 VBB / VPP drivers ports: added none; removed GND
- sheet Status LED drivers ports: added none; removed GND
- sheet USB + reset / boot ports: added none; removed GND
- sheet VBB supply ports: added none; removed GND
- sheet VPP boost supply ports: added none; removed GND
- sheet Vehicle power input ports: added none; removed GND
- sheet Voltage monitoring ports: added none; removed GND

Commit message: Fix scanner protection, ADC isolation and health watchdog
Coordinate the bounded 12 V input clamp and programming FET/capacitor ratings, add powered-off ADC isolation, and supervise the AW9523B permit with a dedicated GPIO13 health heartbeat. Preserve original placements and document all deliberate source-PDF deviations.

Validation: native ERC and full DRC/parity/refill report zero findings; strict preservation/connectivity audit and final adversarial review pass within the documented prototype bounds. Regenerate Rev C PDF, BOM, manufacturing exports, processing sites and verified portable archives. Compatible firmware and bench/mechanical qualification remain required.
Other:
- added sheet Hardware safety + ADC isolation (23_hardware-safety.kicad_sch)
- sheet PCI / J1850 ports: added PCI_VCC; removed +12V
- sheet Voltage monitoring ports: added +12V, V_BA_PRE, V_BT_PRE, V_PR_PRE; removed J1962-16, V_BA, V_BT, V_PR
- note added: "ChryslerScanner V240 | integrated microSD | 277 components | 162 connected nets"
- note removed: "ChryslerScanner V240 | integrated microSD | 259 components | 154 connected nets"

Commit message: Add hook test points and mapped debug access with verified fabrication outputs
Other:
- added sheet Debug access / test points (24_debug-testpoints.kicad_sch)
- note added: "48 hook loops + 4 SPI pads; named global nets"
- note added: "ChryslerScanner V240 | integrated microSD | 329 components incl. 52 test points | 162 connected nets"
- note removed: "ChryslerScanner V240 | integrated microSD | 277 components | 162 connected nets"
