File: projects/chrysler-scanner/current/01_ccd.kicad_sch (KiCad schematic)
At the start: 25 parts, among them Q16 CJ3439KDW, Q7 HSSK8811, U16 TS391C, U17 74LVC1G17, U18 74LVC1G14

Commit message: Finish Chrysler scanner CCD correction and procurement fabrication package
Parts:
- C50, C51, C53: Assembly (none) -> PLACE; MPN (none) -> C0603C221J1GACTU; Manufacturer (none) -> KEMET; Procurement Source (none) -> https://search.kemet.com/component-documentation/download/s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; Selected Voltage Rating (none) -> 100V; Tolerance (none) -> 5%
- C52, C54, C55: Assembly (none) -> PLACE; MPN (none) -> C0603C104K5RACTU; Manufacturer (none) -> KEMET; Procurement Source (none) -> https://search.kemet.com/component-documentation/download/s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; Selected Voltage Rating (none) -> 50V; Tolerance (none) -> 10%
- Q16: footprint footprints:SOT-23-6 -> footprints:SOT-363_SC-70-6_RR; Assembly (none) -> PLACE; MPN (none) -> CJ3439KDW; Manufacturer (none) -> Jiangsu Changjing Electronics Technology; Procurement Source (none) -> https://www.jscj-elec.com/related/23454.html
- Q7: footprint footprints:SOT-23-6 -> footprints:SOT-363_SC-70-6_RR; Assembly (none) -> PLACE; MPN (none) -> HSSK8811; Manufacturer (none) -> HUASHUO Semiconductor; Procurement Source (none) -> https://atta.szlcsc.com/upload/public/pdf/source/20201013/C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
- R100, R101: Assembly (none) -> PLACE; MPN (none) -> CRCW0603360RFKEA; Manufacturer (none) -> Vishay; Procurement Source (none) -> https://www.vishay.com/docs/20035/dcrcwe3.pdf; Selected Power Rating (none) -> 0.1W; Tolerance (none) -> 1%
- R77, R83, R84: Assembly (none) -> PLACE; MPN (none) -> CRCW060310K0FKEA; Manufacturer (none) -> Vishay; Procurement Source (none) -> https://www.vishay.com/docs/20035/dcrcwe3.pdf; Selected Power Rating (none) -> 0.1W; Tolerance (none) -> 1%
- R78, R80: Assembly (none) -> PLACE; MPN (none) -> CRCW060313K0FKEA; Manufacturer (none) -> Vishay; Procurement Source (none) -> https://www.vishay.com/docs/20035/dcrcwe3.pdf; Selected Power Rating (none) -> 0.1W; Tolerance (none) -> 1%
- R79: Assembly (none) -> PLACE; MPN (none) -> CRCW0603120RFKEA; Manufacturer (none) -> Vishay; Procurement Source (none) -> https://www.vishay.com/docs/20035/dcrcwe3.pdf; Selected Power Rating (none) -> 0.1W; Tolerance (none) -> 1%
- R81, R82: Assembly (none) -> PLACE; MPN (none) -> CRCW060310R0FKEA; Manufacturer (none) -> Vishay; Procurement Source (none) -> https://www.vishay.com/docs/20035/dcrcwe3.pdf; Selected Power Rating (none) -> 0.1W; Tolerance (none) -> 1%
- R85, R97: Assembly (none) -> PLACE; MPN (none) -> CRCW06034K70FKEA; Manufacturer (none) -> Vishay; Procurement Source (none) -> https://www.vishay.com/docs/20035/dcrcwe3.pdf; Selected Power Rating (none) -> 0.1W; Tolerance (none) -> 1%
- R98, R99: value 100Ω -> 330Ω; Assembly (none) -> PLACE; MPN (none) -> CRCW0603330RFKEA; Manufacturer (none) -> Vishay; Procurement Source (none) -> https://www.vishay.com/docs/20035/dcrcwe3.pdf; Selected Power Rating (none) -> 0.1W; Tolerance (none) -> 1%
- U16: Assembly (none) -> PLACE; MPN (none) -> TS391ILT; Manufacturer (none) -> STMicroelectronics; Procurement Source (none) -> https://www.st.com/resource/en/datasheet/ts391.pdf
- U17: value 74LVC1G17 -> 74AHCT1G17GV; Assembly (none) -> PLACE; MPN (none) -> 74AHCT1G17GVH; Manufacturer (none) -> Nexperia; Procurement Source (none) -> https://assets.nexperia.com/documents/data-sheet/74AHC_AHCT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
- U18: value 74LVC1G14 -> SN74AHCT1G14; Assembly (none) -> PLACE; MPN (none) -> SN74AHCT1G14DBVR; Manufacturer (none) -> Texas Instruments; Procurement Source (none) -> https://www.ti.com/lit/ds/symlink/sn74ahct1g14.pdf
