File: projects/chrysler-scanner/current/02_pci.kicad_sch (KiCad schematic)
At the start: 12 parts, among them Q1 CJ3439KDW, U9 TS391C

Commit message: Fix scanner protection, ADC isolation and health watchdog
Coordinate the bounded 12 V input clamp and programming FET/capacitor ratings, add powered-off ADC isolation, and supervise the AW9523B permit with a dedicated GPIO13 health heartbeat. Preserve original placements and document all deliberate source-PDF deviations.

Validation: native ERC and full DRC/parity/refill report zero findings; strict preservation/connectivity audit and final adversarial review pass within the documented prototype bounds. Regenerate Rev C PDF, BOM, manufacturing exports, processing sites and verified portable archives. Compatible firmware and bench/mechanical qualification remain required.
Connections:
- net +12V renamed PCI_VCC

Commit message: Finish Chrysler scanner CCD correction and procurement fabrication package
Parts:
- C11: Assembly (none) -> PLACE; MPN (none) -> C1206C104K1RACTU; Manufacturer (none) -> KEMET; Procurement Source (none) -> https://search.kemet.com/component-documentation/download/s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; Selected Voltage Rating (none) -> 100V; Tolerance (none) -> 10%
- C12: Assembly (none) -> PLACE; MPN (none) -> C1206C221J1GACTU; Manufacturer (none) -> KEMET; Procurement Source (none) -> https://search.kemet.com/component-documentation/download/s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; Selected Voltage Rating (none) -> 100V; Tolerance (none) -> 5%
- Q1: footprint footprints:SOT-23-6 -> footprints:SOT-363_SC-70-6_RR; Assembly (none) -> PLACE; MPN (none) -> CJ3439KDW; Manufacturer (none) -> Jiangsu Changjing Electronics Technology; Procurement Source (none) -> https://www.jscj-elec.com/related/23454.html
- R18, R21, R6: Assembly (none) -> PLACE; MPN (none) -> CRCW060310K0FKEA; Manufacturer (none) -> Vishay; Procurement Source (none) -> https://www.vishay.com/docs/20035/dcrcwe3.pdf; Selected Power Rating (none) -> 0.1W; Tolerance (none) -> 1%
- R19: Assembly (none) -> PLACE; MPN (none) -> CRCW1206360RFKEA; Manufacturer (none) -> Vishay; Procurement Source (none) -> https://www.vishay.com/docs/20035/dcrcwe3.pdf; Selected Power Rating (none) -> 0.25W; Tolerance (none) -> 1%
- R20: Assembly (none) -> PLACE; MPN (none) -> CRCW12061K00FKEA; Manufacturer (none) -> Vishay; Procurement Source (none) -> https://www.vishay.com/docs/20035/dcrcwe3.pdf; Selected Power Rating (none) -> 0.25W; Tolerance (none) -> 1%
- R4: Assembly (none) -> PLACE; MPN (none) -> CRCW06032K00FKEA; Manufacturer (none) -> Vishay; Procurement Source (none) -> https://www.vishay.com/docs/20035/dcrcwe3.pdf; Selected Power Rating (none) -> 0.1W; Tolerance (none) -> 1%
- R5, R7: Assembly (none) -> PLACE; MPN (none) -> CRCW06034K70FKEA; Manufacturer (none) -> Vishay; Procurement Source (none) -> https://www.vishay.com/docs/20035/dcrcwe3.pdf; Selected Power Rating (none) -> 0.1W; Tolerance (none) -> 1%
- U9: Assembly (none) -> PLACE; MPN (none) -> TS391ILT; Manufacturer (none) -> STMicroelectronics; Procurement Source (none) -> https://www.st.com/resource/en/datasheet/ts391.pdf
