File: projects/chrysler-scanner/current/04_sci-6-12.kicad_sch (KiCad schematic)
At the start: 12 parts, among them Q2 2N7002DW, Q6 CJ3439KDW, U13 74LVC2G66

Commit message: Finish Chrysler scanner CCD correction and procurement fabrication package
Parts:
- C38: Assembly (none) -> PLACE; MPN (none) -> C0603C104K5RACTU; Manufacturer (none) -> KEMET; Procurement Source (none) -> https://search.kemet.com/component-documentation/download/s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; Selected Voltage Rating (none) -> 50V; Tolerance (none) -> 10%
- Q2: value 2N7002DW -> DMN62D2UDM; Assembly (none) -> PLACE; MPN (none) -> DMN62D2UDM-7; Manufacturer (none) -> Diodes Incorporated; Procurement Source (none) -> https://www.diodes.com/datasheet/download/DMN62D2UDM.pdf
- Q6: footprint footprints:SOT-23-6 -> footprints:SOT-363_SC-70-6_RR; Assembly (none) -> PLACE; MPN (none) -> CJ3439KDW; Manufacturer (none) -> Jiangsu Changjing Electronics Technology; Procurement Source (none) -> https://www.jscj-elec.com/related/23454.html
- R29, R30, R33: Assembly (none) -> PLACE; MPN (none) -> CRCW12064K70FKEA; Manufacturer (none) -> Vishay; Procurement Source (none) -> https://www.vishay.com/docs/20035/dcrcwe3.pdf; Selected Power Rating (none) -> 0.25W; Tolerance (none) -> 1%
- R31, R34, R75: Assembly (none) -> PLACE; MPN (none) -> CRCW060310K0FKEA; Manufacturer (none) -> Vishay; Procurement Source (none) -> https://www.vishay.com/docs/20035/dcrcwe3.pdf; Selected Power Rating (none) -> 0.1W; Tolerance (none) -> 1%
- R32, R76: Assembly (none) -> PLACE; MPN (none) -> CRCW06034K70FKEA; Manufacturer (none) -> Vishay; Procurement Source (none) -> https://www.vishay.com/docs/20035/dcrcwe3.pdf; Selected Power Rating (none) -> 0.1W; Tolerance (none) -> 1%
- U13: Assembly (none) -> PLACE; MPN (none) -> SN74LVC2G66DCTR; Manufacturer (none) -> Texas Instruments; Procurement Source (none) -> https://www.ti.com/lit/ds/symlink/sn74lvc2g66.pdf
