File: projects/chrysler-scanner/current/06_obd-protection.kicad_sch (KiCad schematic)
At the start: 12 parts, among them J1 226A-1202

Commit message: Finish Chrysler scanner CCD correction and procurement fabrication package
Parts:
- C25, C36, C37, C39, C40, C42, C44: Assembly (none) -> PLACE; MPN (none) -> C0603C221J1GACTU; Manufacturer (none) -> KEMET; Procurement Source (none) -> https://search.kemet.com/component-documentation/download/s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; Selected Voltage Rating (none) -> 100V; Tolerance (none) -> 5%
- D11: value MSK4005 -> PMEG4005; Assembly (none) -> PLACE; MPN (none) -> PMEG4005EGWX; Manufacturer (none) -> Nexperia; Procurement Source (none) -> https://assets.nexperia.com/documents/data-sheet/PMEG4005EG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
- D12, D13, D14: value ESD5Z12V -> SMF12A; Assembly (none) -> PLACE; MPN (none) -> SMF12A; Manufacturer (none) -> Diotec Semiconductor; Procurement Source (none) -> https://diotec.com/en/product/SMF12A.html
- J1: Assembly (none) -> PLACE; MPN (none) -> 226A-1202; Manufacturer (none) -> ATTEND; Procurement Source (none) -> https://www.attend.com.tw/data/download/file/226A-1202.pdf
Changed lines of the file:
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@@
 			)
 		)
-		(property "Datasheet" ""
+		(property "Datasheet" "https://search.kemet.com/component-documentation/download/specsheet/C0603C221J1GACTU"
 			(at 137.16000 53.34000 0)
 			(hide yes)
@@
 			)
 		)
-	)
+(property "Manufacturer" "KEMET" (at 0 0 0) (effects (font (size 1 1)) (hide yes)))
+(property "MPN" "C0603C221J1GACTU" (at 0 0 0) (effects (font (size 1 1)) (hide yes)))
+(property "Procurement Source" "https://search.kemet.com/component-documentation/download/specsheet/C0603C221J1GACTU" (at 0 0 0) (effects (font (size 1 1)) (hide yes)))
+(property "Assembly" "PLACE" (at 0 0 0) (effects (font (size 1 1)) (hide yes)))
+(property "Selected Voltage Rating" "100V" (at 0 0 0) (effects (font (size 1 1)) (hide yes)))
+(property "Tolerance" "5%" (at 0 0 0) (effects (font (size 1 1)) (hide yes)))
+)
 	(symbol
 		(lib_id "ChryslerScanner:D11")
@@
 			)
 		)
-		(property "Value" "MSK4005"
+		(property "Value" "PMEG4005"
 			(at 34.04740 51.75000 0)
 			(show_name no)
@@
 			)
 		)
-		(property "Datasheet" ""
+		(property "Datasheet" "https://assets.nexperia.com/documents/data-sheet/PMEG4005EGW.pdf"
 			(at 25.40000 50.80000 0)
 			(hide yes)
@@
 			)
 		)
-	)
+(property "Manufacturer" "Nexperia" (at 0 0 0) (effects (font (size 1 1)) (hide yes)))
+(property "MPN" "PMEG4005EGWX" (at 0 0 0) (effects (font (size 1 1)) (hide yes)))
+(property "Procurement Source" "https://assets.nexperia.com/documents/data-sheet/PMEG4005EGW.pdf" (at 0 0 0) (effects (font (size 1 1)) (hide yes)))
+(property "Assembly" "PLACE" (at 0 0 0) (effects (font (size 1 1)) (hide yes)))
+)
 	(symbol
 		(lib_id "power:GND")
@@
 			)
 		)
-		(property "Value" "ESD5Z12V"
+		(property "Value" "SMF12A"
 			(at 75.18630 72.07000 0)
 			(show_name no)
@@
 			)
 		)
-		(property "Datasheet" ""
+		(property "Datasheet" "https://diotec.com/en/product/SMF12A.html"
 			(at 66.04000 71.12000 0)
 			(hide yes)
@@
 			)
 		)
-	)
+(property "Manufacturer" "Diotec Semiconductor" (at 0 0 0) (effects (font (size 1 1)) (hide yes)))
+(property "MPN" "SMF12A" (at 0 0 0) (effects (font (size 1 1)) (hide yes)))
+(property "Procurement Source" "https://diotec.com/en/product/SMF12A.html" (at 0 0 0) (effects (font (size 1 1)) (hide yes)))
+(property "Assembly" "PLACE" (at 0 0 0) (effects (font (size 1 1)) (hide yes)))
+)
 	(symbol
 		(lib_id "power:GND")
@@
 			)
 		)
-		(property "Datasheet" ""
+		(property "Datasheet" "https://search.kemet.com/component-documentation/download/specsheet/C0603C221J1GACTU"
 			(at 205.74000 53.34 0)
 			(hide yes)
@@
 			)
 		)
-	)
+(property "Manufacturer" "KEMET" (at 0 0 0) (effects (font (size 1 1)) (hide yes)))
+(property "MPN" "C0603C221J1GACTU" (at 0 0 0) (effects (font (size 1 1)) (hide yes)))
+(property "Procurement Source" "https://search.kemet.com/component-documentation/download/specsheet/C0603C221J1GACTU" (at 0 0 0) (effects (font (size 1 1)) (hide yes)))
+(property "Assembly" "PLACE" (at 0 0 0) (effects (font (size 1 1)) (hide yes)))
+(property "Selected Voltage Rating" "100V" (at 0 0 0) (effects (font (size 1 1)) (hide yes)))
+(property "Tolerance" "5%" (at 0 0 0) (effects (font (size 1 1)) (hide yes)))
+)
 	(symbol
 		(lib_id "ChryslerScanner:C36")
@@
 			)
 		)
-		(property "Datasheet" ""
+		(property "Datasheet" "https://search.kemet.com/component-documentation/download/specsheet/C0603C221J1GACTU"
 			(at 109.22000 53.34000 0)
 			(hide yes)
@@
 			)
 		)
-	)
+(property "Manufacturer" "KEMET" (at 0 0 0) (effects (font (size 1 1)) (hide yes)))
+(property "MPN" "C0603C221J1GACTU" (at 0 0 0) (effects (font (size 1 1)) (hide yes)))
+(property "Procurement Source" "https://search.kemet.com/component-documentation/download/specsheet/C0603C221J1GACTU" (at 0 0 0) (effects (font (size 1 1)) (hide yes)))
+(property "Assembly" "PLACE" (at 0 0 0) (effects (font (size 1 1)) (hide yes)))
+(property "Selected Voltage Rating" "100V" (at 0 0 0) (effects (font (size 1 1)) (hide yes)))
+(property "Tolerance" "5%" (at 0 0 0) (effects (font (size 1 1)) (hide yes)))
+)
 	(symbol
 		(lib_id "power:GND")
@@
 			)
 		)
-		(property "Datasheet" ""
+		(property "Datasheet" "https://www.attend.com.tw/data/download/file/226A-1202.pdf"
 			(at 66.04 191.77 0)
 			(hide yes)
@@
 			)
 		)
-	)
+(property "Manufacturer" "ATTEND" (at 0 0 0) (effects (font (size 1 1)) (hide yes)))
+(property "MPN" "226A-1202" (at 0 0 0) (effects (font (size 1 1)) (hide yes)))
+(property "Procurement Source" "https://www.attend.com.tw/data/download/file/226A-1202.pdf" (at 0 0 0) (effects (font (size 1 1)) (hide yes)))
+(property "Assembly" "PLACE" (at 0 0 0) (effects (font (size 1 1)) (hide yes)))
+)
 	(symbol
 		(lib_id "ChryslerScanner:C39")
@@
 			)
 		)
-		(property "Datasheet" ""
+		(property "Datasheet" "https://search.kemet.com/component-documentation/download/specsheet/C0603C221J1GACTU"
 			(at 177.80000 53.34000 0)
 			(hide yes)
@@
 			)
 		)
-	)
+(property "Manufacturer" "KEMET" (at 0 0 0) (effects (font (size 1 1)) (hide yes)))
+(property "MPN" "C0603C221J1GACTU" (at 0 0 0) (effects (font (size 1 1)) (hide yes)))
+(property "Procurement Source" "https://search.kemet.com/component-documentation/download/specsheet/C0603C221J1GACTU" (at 0 0 0) (effects (font (size 1 1)) (hide yes)))
+(property "Assembly" "PLACE" (at 0 0 0) (effects (font (size 1 1)) (hide yes)))
+(property "Selected Voltage Rating" "100V" (at 0 0 0) (effects (font (size 1 1)) (hide yes)))
+(property "Tolerance" "5%" (at 0 0 0) (effects (font (size 1 1)) (hide yes)))
+)
 	(symbol
 		(lib_id "power:GND")
@@
 			)
 		)
-		(property "Datasheet" ""
+		(property "Datasheet" "https://search.kemet.com/component-documentation/download/specsheet/C0603C221J1GACTU"
 			(at 35.56000 116.84000 0)
 			(hide yes)
@@
 			)
 		)
-	)
+(property "Manufacturer" "KEMET" (at 0 0 0) (effects (font (size 1 1)) (hide yes)))
+(property "MPN" "C0603C221J1GACTU" (at 0 0 0) (effects (font (size 1 1)) (hide yes)))
+(property "Procurement Source" "https://search.kemet.com/component-documentation/download/specsheet/C0603C221J1GACTU" (at 0 0 0) (effects (font (size 1 1)) (hide yes)))
+(property "Assembly" "PLACE" (at 0 0 0) (effects (font (size 1 1)) (hide yes)))
+(property "Selected Voltage Rating" "100V" (at 0 0 0) (effects (font (size 1 1)) (hide yes)))
+(property "Tolerance" "5%" (at 0 0 0) (effects (font (size 1 1)) (hide yes)))
+)
 	(symbol
 		(lib_id "ChryslerScanner:D14")
@@
 			)
 		)
-		(property "Value" "ESD5Z12V"
+		(property "Value" "SMF12A"
 			(at 189.48630 117.79000 0)
 			(show_name no)
@@
 			)
 		)
-		(property "Datasheet" ""
+		(property "Datasheet" "https://diotec.com/en/product/SMF12A.html"
 			(at 180.34000 116.84000 0)
 			(hide yes)
@@
 			)
 		)
-	)
+(property "Manufacturer" "Diotec Semiconductor" (at 0 0 0) (effects (font (size 1 1)) (hide yes)))
+(property "MPN" "SMF12A" (at 0 0 0) (effects (font (size 1 1)) (hide yes)))
+(property "Procurement Source" "https://diotec.com/en/product/SMF12A.html" (at 0 0 0) (effects (font (size 1 1)) (hide yes)))
+(property "Assembly" "PLACE" (at 0 0 0) (effects (font (size 1 1)) (hide yes)))
+)
 	(symbol
 		(lib_id "power:GND")
@@
 			)
 		)
-		(property "Datasheet" ""
+		(property "Datasheet" "https://search.kemet.com/component-documentation/download/specsheet/C0603C221J1GACTU"
 			(at 45.72000 71.12000 0)
 			(hide yes)
@@
 			)
 		)
-	)
+(property "Manufacturer" "KEMET" (at 0 0 0) (effects (font (size 1 1)) (hide yes)))
+(property "MPN" "C0603C221J1GACTU" (at 0 0 0) (effects (font (size 1 1)) (hide yes)))
+(property "Procurement Source" "https://search.kemet.com/component-documentation/download/specsheet/C0603C221J1GACTU" (at 0 0 0) (effects (font (size 1 1)) (hide yes)))
+(property "Assembly" "PLACE" (at 0 0 0) (effects (font (size 1 1)) (hide yes)))
+(property "Selected Voltage Rating" "100V" (at 0 0 0) (effects (font (size 1 1)) (hide yes)))
+(property "Tolerance" "5%" (at 0 0 0) (effects (font (size 1 1)) (hide yes)))
+)
 	(symbol
 		(lib_id "ChryslerScanner:C44")
@@
 			)
 		)
-		(property "Datasheet" ""
+		(property "Datasheet" "https://search.kemet.com/component-documentation/download/specsheet/C0603C221J1GACTU"
 			(at 78.74000 116.84000 0)
 			(hide yes)
@@
 			)
 		)
-	)
+(property "Manufacturer" "KEMET" (at 0 0 0) (effects (font (size 1 1)) (hide yes)))
+(property "MPN" "C0603C221J1GACTU" (at 0 0 0) (effects (font (size 1 1)) (hide yes)))
+(property "Procurement Source" "https://search.kemet.com/component-documentation/download/specsheet/C0603C221J1GACTU" (at 0 0 0) (effects (font (size 1 1)) (hide yes)))
+(property "Assembly" "PLACE" (at 0 0 0) (effects (font (size 1 1)) (hide yes)))
+(property "Selected Voltage Rating" "100V" (at 0 0 0) (effects (font (size 1 1)) (hide yes)))
+(property "Tolerance" "5%" (at 0 0 0) (effects (font (size 1 1)) (hide yes)))
+)
 	(symbol
 		(lib_id "ChryslerScanner:D13")
@@
 			)
 		)
-		(property "Value" "ESD5Z12V"
+		(property "Value" "SMF12A"
 			(at 141.22630 117.79000 0)
 			(show_name no)
@@
 			)
 		)
-		(property "Datasheet" ""
+		(property "Datasheet" "https://diotec.com/en/product/SMF12A.html"
 			(at 132.08000 116.84000 0)
 			(hide yes)
@@
 			)
 		)
-	)
+(property "Manufacturer" "Diotec Semiconductor" (at 0 0 0) (effects (font (size 1 1)) (hide yes)))
+(property "MPN" "SMF12A" (at 0 0 0) (effects (font (size 1 1)) (hide yes)))
+(property "Procurement Source" "https://diotec.com/en/product/SMF12A.html" (at 0 0 0) (effects (font (size 1 1)) (hide yes)))
+(property "Assembly" "PLACE" (at 0 0 0) (effects (font (size 1 1)) (hide yes)))
+)
 	(symbol
 		(lib_id "power:GND")
