File: projects/chrysler-scanner/current/07_vehicle-input.kicad_sch (KiCad schematic)
At the start: 4 parts

Commit message: Fix scanner protection, ADC isolation and health watchdog
Coordinate the bounded 12 V input clamp and programming FET/capacitor ratings, add powered-off ADC isolation, and supervise the AW9523B permit with a dedicated GPIO13 health heartbeat. Preserve original placements and document all deliberate source-PDF deviations.

Validation: native ERC and full DRC/parity/refill report zero findings; strict preservation/connectivity audit and final adversarial review pass within the documented prototype bounds. Regenerate Rev C PDF, BOM, manufacturing exports, processing sites and verified portable archives. Compatible firmware and bench/mechanical qualification remain required.
Parts:
- C1: Voltage Rating (none) -> 50V
- D1: value SMBJ30CA -> SMBJ16CA

Commit message: Restore schematic polarity and visible capacitor ratings
Changed lines of the file:
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@@
 			)
 		)
-	(property "Voltage Rating" "50V" (at 0 0 0) (effects (font (size 1 1)) (hide yes))))
+	(property "Voltage Rating" "50V" (at 65.0445 86.87 0) (effects (font (size 1 1)))))
 	(symbol
 		(lib_id "ChryslerScanner:D2")

Commit message: Finish Chrysler scanner CCD correction and procurement fabrication package
Parts:
- C1: Assembly (none) -> PLACE; MPN (none) -> UPW1H101MPD; Manufacturer (none) -> Nichicon; Procurement Source (none) -> https://www.nichicon.co.jp/english/series_items/catalog_pdf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; Selected Height (none) -> 11.5mm; Selected Voltage Rating (none) -> 50V; Tolerance (none) -> 20%
- D1: Assembly (none) -> PLACE; MPN (none) -> SMBJ16CA; Manufacturer (none) -> Littelfuse; Procurement Source (none) -> https://www.littelfuse.com/products/overvoltage-protection/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
- D2: Assembly (none) -> PLACE; MPN (none) -> SS56-E3/57T; Manufacturer (none) -> Vishay; Procurement Source (none) -> https://www.vishay.com/docs/88714/ss52.pdf
- JP1: Assembly (none) -> PCB_FEATURE_CLOSED; MPN (none) -> SOLDER_BRIDGE_NO_COMPONENT; Manufacturer (none) -> PCB feature; Procurement Source (none) -> KiCad native solder jumper
Changed lines of the file:
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@@
 			)
 		)
-	)
+(property "Manufacturer" "PCB feature" (at 0 0 0) (effects (font (size 1 1)) (hide yes)))
+(property "MPN" "SOLDER_BRIDGE_NO_COMPONENT" (at 0 0 0) (effects (font (size 1 1)) (hide yes)))
+(property "Procurement Source" "KiCad native solder jumper" (at 0 0 0) (effects (font (size 1 1)) (hide yes)))
+(property "Assembly" "PCB_FEATURE_CLOSED" (at 0 0 0) (effects (font (size 1 1)) (hide yes)))
+)
 	(symbol
 		(lib_id "power:GND")
@@
 			)
 		)
-		(property "Datasheet" ""
+		(property "Datasheet" "https://www.littelfuse.com/products/overvoltage-protection/tvs-diodes/smbj/smbj16ca"
 			(at 20.32 83.82 0)
 			(hide yes)
@@
 			)
 		)
-	)
+(property "Manufacturer" "Littelfuse" (at 0 0 0) (effects (font (size 1 1)) (hide yes)))
+(property "MPN" "SMBJ16CA" (at 0 0 0) (effects (font (size 1 1)) (hide yes)))
+(property "Procurement Source" "https://www.littelfuse.com/products/overvoltage-protection/tvs-diodes/smbj/smbj16ca" (at 0 0 0) (effects (font (size 1 1)) (hide yes)))
+(property "Assembly" "PLACE" (at 0 0 0) (effects (font (size 1 1)) (hide yes)))
+)
 	(symbol
 		(lib_id "ChryslerScanner:C1")
@@
 			)
 		)
-		(property "Datasheet" ""
+		(property "Datasheet" "https://www.nichicon.co.jp/english/series_items/catalog_pdf/e-upw.pdf"
 			(at 55.88 83.82 0)
 			(hide yes)
@@
 			)
 		)
-	(property "Voltage Rating" "50V" (at 65.0445 86.87 0) (effects (font (size 1 1)))))
+	(property "Voltage Rating" "50V" (at 65.0445 86.87 0) (effects (font (size 1 1))))
+(property "Manufacturer" "Nichicon" (at 0 0 0) (effects (font (size 1 1)) (hide yes)))
+(property "MPN" "UPW1H101MPD" (at 0 0 0) (effects (font (size 1 1)) (hide yes)))
+(property "Procurement Source" "https://www.nichicon.co.jp/english/series_items/catalog_pdf/e-upw.pdf" (at 0 0 0) (effects (font (size 1 1)) (hide yes)))
+(property "Assembly" "PLACE" (at 0 0 0) (effects (font (size 1 1)) (hide yes)))
+(property "Selected Voltage Rating" "50V" (at 0 0 0) (effects (font (size 1 1)) (hide yes)))
+(property "Tolerance" "20%" (at 0 0 0) (effects (font (size 1 1)) (hide yes)))
+(property "Selected Height" "11.5mm" (at 0 0 0) (effects (font (size 1 1)) (hide yes)))
+)
 	(symbol
 		(lib_id "ChryslerScanner:D2")
@@
 			)
 		)
-		(property "Datasheet" ""
+		(property "Datasheet" "https://www.vishay.com/docs/88714/ss52.pdf"
 			(at 38.1 60.96 0)
 			(hide yes)
@@
 			)
 		)
-	)
-)
+(property "Manufacturer" "Vishay" (at 0 0 0) (effects (font (size 1 1)) (hide yes)))
+(property "MPN" "SS56-E3/57T" (at 0 0 0) (effects (font (size 1 1)) (hide yes)))
+(property "Procurement Source" "https://www.vishay.com/docs/88714/ss52.pdf" (at 0 0 0) (effects (font (size 1 1)) (hide yes)))
+(property "Assembly" "PLACE" (at 0 0 0) (effects (font (size 1 1)) (hide yes)))
+)
+)
