File: projects/chrysler-scanner/current/16_mcu.kicad_sch (KiCad schematic)
At the start: 16 parts, among them U10 ESP32-PICO-V3-02

Commit message: Fix scanner protection, ADC isolation and health watchdog
Coordinate the bounded 12 V input clamp and programming FET/capacitor ratings, add powered-off ADC isolation, and supervise the AW9523B permit with a dedicated GPIO13 health heartbeat. Preserve original placements and document all deliberate source-PDF deviations.

Validation: native ERC and full DRC/parity/refill report zero findings; strict preservation/connectivity audit and final adversarial review pass within the documented prototype bounds. Regenerate Rev C PDF, BOM, manufacturing exports, processing sites and verified portable archives. Compatible firmware and bench/mechanical qualification remain required.
Parts:
- C26, C27: Voltage Rating (none) -> 10V

Commit message: Restore schematic polarity and visible capacitor ratings
Changed lines of the file:
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@@
 			)
 		)
-	(property "Voltage Rating" "10V" (at 0 0 0) (effects (font (size 1 1)) (hide yes))))
+	(property "Voltage Rating" "10V" (at 19.8641 74.17 0) (effects (font (size 1 1)))))
 	(symbol
 		(lib_id "ChryslerScanner:C31")
@@
 			)
 		)
-	(property "Voltage Rating" "10V" (at 0 0 0) (effects (font (size 1 1)) (hide yes))))
+	(property "Voltage Rating" "10V" (at 51.2559 79.25 0) (effects (font (size 1 1)))))
 	(symbol
 		(lib_id "ChryslerScanner:C29")

Commit message: Finish Chrysler scanner CCD correction and procurement fabrication package
Parts:
- AE1: Assembly (none) -> PLACE; MPN (none) -> ANT3216LL00R2400A; Manufacturer (none) -> Walsin; Procurement Source (none) -> https://www.passivecomponent.com/antenna/
- C26, C27, C28: Assembly (none) -> PLACE; MPN (none) -> C1608X5R1A106K080AC; Manufacturer (none) -> TDK; Procurement Source (none) -> https://product.tdk.com/en/search/capacitor/ceramic/mlcc/in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; Selected Voltage Rating (none) -> 10V; Tolerance (none) -> 10%
- C29, C30, C31, C32, C33, C46: Assembly (none) -> PLACE; MPN (none) -> C0603C104K5RACTU; Manufacturer (none) -> KEMET; Procurement Source (none) -> https://search.kemet.com/component-documentation/download/s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; Selected Voltage Rating (none) -> 50V; Tolerance (none) -> 10%
- C45: Assembly (none) -> PLACE; MPN (none) -> C0603C105K4RACTU; Manufacturer (none) -> KEMET; Procurement Source (none) -> https://search.kemet.com/component-documentation/download/s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; Selected Voltage Rating (none) -> 16V; Tolerance (none) -> 10%
- R22: Assembly (none) -> PLACE; MPN (none) -> CRCW06030000Z0EA; Manufacturer (none) -> Vishay; Procurement Source (none) -> https://www.vishay.com/docs/20035/dcrcwe3.pdf; Selected Power Rating (none) -> 0.1W; Tolerance (none) -> jumper
- R23, R24: Assembly (none) -> DNP; MPN (none) -> DNP_RF_TUNING; Manufacturer (none) -> Not fitted; Procurement Source (none) -> RF tuning pads intentionally unpopulated
- R48: Assembly (none) -> PLACE; MPN (none) -> CRCW060310K0FKEA; Manufacturer (none) -> Vishay; Procurement Source (none) -> https://www.vishay.com/docs/20035/dcrcwe3.pdf; Selected Power Rating (none) -> 0.1W; Tolerance (none) -> 1%
- U10: Assembly (none) -> PLACE; MPN (none) -> ESP32-PICO-V3-02; Manufacturer (none) -> Espressif; Procurement Source (none) -> https://www.espressif.com/sites/default/files/documentation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
