File: projects/chrysler-scanner/current/19_usb.kicad_sch (KiCad schematic)
At the start: 19 parts, among them J2 USB-C, Q5 UMH3N, SW1 RESET, SW2 BOOT, U1 SY6283, U11 USBLC6-2SC6, U12 CP2102

Commit message: Fix scanner protection, ADC isolation and health watchdog
Coordinate the bounded 12 V input clamp and programming FET/capacitor ratings, add powered-off ADC isolation, and supervise the AW9523B permit with a dedicated GPIO13 health heartbeat. Preserve original placements and document all deliberate source-PDF deviations.

Validation: native ERC and full DRC/parity/refill report zero findings; strict preservation/connectivity audit and final adversarial review pass within the documented prototype bounds. Regenerate Rev C PDF, BOM, manufacturing exports, processing sites and verified portable archives. Compatible firmware and bench/mechanical qualification remain required.
Parts:
- C35: Voltage Rating (none) -> 10V

Commit message: Restore schematic polarity and visible capacitor ratings
Changed lines of the file:
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@@
 			)
 		)
-	(property "Voltage Rating" "10V" (at 0 0 0) (effects (font (size 1 1)) (hide yes))))
+	(property "Voltage Rating" "10V" (at 376.376 132.59 0) (effects (font (size 1 1)))))
 	(symbol
 		(lib_id "ChryslerScanner:Q5")

Commit message: Finish Chrysler scanner CCD correction and procurement fabrication package
Parts:
- C2, C3: Assembly (none) -> PLACE; MPN (none) -> CGA5L1X7R1H106K160AC; Manufacturer (none) -> TDK; Procurement Source (none) -> https://product.tdk.com/info/en/documents/chara_sheet/CGA5L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; Selected Voltage Rating (none) -> 50V; Tolerance (none) -> 10%
- C34: Assembly (none) -> PLACE; MPN (none) -> C0603C104K5RACTU; Manufacturer (none) -> KEMET; Procurement Source (none) -> https://search.kemet.com/component-documentation/download/s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; Selected Voltage Rating (none) -> 50V; Tolerance (none) -> 10%
- C35: Assembly (none) -> PLACE; MPN (none) -> C1608X5R1A106K080AC; Manufacturer (none) -> TDK; Procurement Source (none) -> https://product.tdk.com/en/search/capacitor/ceramic/mlcc/in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; Selected Voltage Rating (none) -> 10V; Tolerance (none) -> 10%
- D3: Assembly (none) -> PLACE; MPN (none) -> LMBR130T1G; Manufacturer (none) -> onsemi; Procurement Source (none) -> https://www.onsemi.com/pdf/datasheet/lmbr130t1-d.pdf
- J2: Assembly (none) -> PLACE; MPN (none) -> USB4105-GF-A; Manufacturer (none) -> GCT; Procurement Source (none) -> https://gct.co/connector/usb4105
- JP2: Assembly (none) -> PCB_FEATURE_OPEN; MPN (none) -> SOLDER_BRIDGE_NO_COMPONENT; Manufacturer (none) -> PCB feature; Procurement Source (none) -> KiCad native solder jumper
- Q5: Assembly (none) -> PLACE; MPN (none) -> UMH3NTR; Manufacturer (none) -> ROHM; Procurement Source (none) -> https://fscdn.rohm.com/en/products/databook/datasheet/discr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
- R102, R103: Assembly (none) -> PLACE; MPN (none) -> CRCW06035K10FKEA; Manufacturer (none) -> Vishay; Procurement Source (none) -> https://www.vishay.com/docs/20035/dcrcwe3.pdf; Selected Power Rating (none) -> 0.1W; Tolerance (none) -> 1%
- R25: Assembly (none) -> PLACE; MPN (none) -> CRCW0603499RFKEA; Manufacturer (none) -> Vishay; Procurement Source (none) -> https://www.vishay.com/docs/20035/dcrcwe3.pdf; Selected Power Rating (none) -> 0.1W; Tolerance (none) -> 1%
- R26: Assembly (none) -> PLACE; MPN (none) -> CRCW060322K0FKEA; Manufacturer (none) -> Vishay; Procurement Source (none) -> https://www.vishay.com/docs/20035/dcrcwe3.pdf; Selected Power Rating (none) -> 0.1W; Tolerance (none) -> 1%
- R27: Assembly (none) -> PLACE; MPN (none) -> CRCW060347K0FKEA; Manufacturer (none) -> Vishay; Procurement Source (none) -> https://www.vishay.com/docs/20035/dcrcwe3.pdf; Selected Power Rating (none) -> 0.1W; Tolerance (none) -> 1%
- R28: Assembly (none) -> PLACE; MPN (none) -> CRCW06034K70FKEA; Manufacturer (none) -> Vishay; Procurement Source (none) -> https://www.vishay.com/docs/20035/dcrcwe3.pdf; Selected Power Rating (none) -> 0.1W; Tolerance (none) -> 1%
- SW1, SW2: Assembly (none) -> PLACE; MPN (none) -> TL3305AF160QG; Manufacturer (none) -> E-Switch; Procurement Source (none) -> https://www.e-switch.com/wp-content/uploads/2023/01/TL3305.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
- U1: Assembly (none) -> PLACE; MPN (none) -> SY6283DRC; Manufacturer (none) -> Silergy; Procurement Source (none) -> https://www.silergy.com/zh/download/downloadFile?ftype=note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
- U11: Assembly (none) -> PLACE; MPN (none) -> USBLC6-2SC6; Manufacturer (none) -> STMicroelectronics; Procurement Source (none) -> https://www.st.com/resource/en/datasheet/usblc6-2.pdf
- U12: Assembly (none) -> PLACE; MPN (none) -> CP2102-GMR; Manufacturer (none) -> Silicon Labs; Procurement Source (none) -> https://www.silabs.com/documents/public/data-sheets/CP2102-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
