File: projects/chrysler-scanner/current/23_hardware-safety.kicad_sch (KiCad schematic)
At the start: 18 parts, among them U21 TMUX1511PWR, U22 LTC6993HS6-2#TRMPBF, U23 SN74LVC1G11DBVR, U24 TLV803EA30DBZR

Commit message: Finish Chrysler scanner CCD correction and procurement fabrication package
Parts:
- C62, C63, C64, C65: Assembly (none) -> PLACE; MPN (none) -> C0603C104K5RACTU; Manufacturer (none) -> KEMET; Procurement Source (none) -> https://search.kemet.com/component-documentation/download/s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; Selected Voltage Rating (none) -> 50V; Tolerance (none) -> 10%
- D30: Assembly (none) -> PLACE; MPN (none) -> BZT52H-B15,115; Manufacturer (none) -> Nexperia; Procurement Source (none) -> https://assets.nexperia.com/documents/data-sheet/BZT52H_SER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
- R115: Assembly (none) -> PLACE; MPN (none) -> TNPW0603100KBEEA; Manufacturer (none) -> Vishay; Procurement Source (none) -> https://www.vishay.com/docs/28758/tnpw_e3.pdf; Selected Power Rating (none) -> 0.1W; Tolerance (none) -> 0.1%
- R116: Assembly (none) -> PLACE; MPN (none) -> CRCW0603191KFKEA; Manufacturer (none) -> Vishay; Procurement Source (none) -> https://www.vishay.com/docs/20035/dcrcwe3.pdf; Selected Power Rating (none) -> 0.1W; Tolerance (none) -> 1%
- R117, R120, R121, R122: Assembly (none) -> PLACE; MPN (none) -> CRCW0603100KFKEA; Manufacturer (none) -> Vishay; Procurement Source (none) -> https://www.vishay.com/docs/20035/dcrcwe3.pdf; Selected Power Rating (none) -> 0.1W; Tolerance (none) -> 1%
- R118, R119: Assembly (none) -> PLACE; MPN (none) -> CRCW060310K0FKEA; Manufacturer (none) -> Vishay; Procurement Source (none) -> https://www.vishay.com/docs/20035/dcrcwe3.pdf; Selected Power Rating (none) -> 0.1W; Tolerance (none) -> 1%
- R123: Assembly (none) -> PLACE; MPN (none) -> CRCW25121K00FKEA; Manufacturer (none) -> Vishay; Procurement Source (none) -> https://www.vishay.com/docs/20035/dcrcwe3.pdf; Selected Power Rating (none) -> 1W; Tolerance (none) -> 1%
- U21: Assembly (none) -> PLACE; MPN (none) -> TMUX1511PWR; Manufacturer (none) -> Texas Instruments; Procurement Source (none) -> https://www.ti.com/lit/ds/symlink/tmux1511.pdf
- U22: Assembly (none) -> PLACE; MPN (none) -> LTC6993HS6-2#TRMPBF; Manufacturer (none) -> Analog Devices; Procurement Source (none) -> https://www.analog.com/media/en/technical-documentation/dat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
- U23: Assembly (none) -> PLACE; MPN (none) -> SN74LVC1G11DBVR; Manufacturer (none) -> Texas Instruments; Procurement Source (none) -> https://www.ti.com/lit/ds/symlink/sn74lvc1g11.pdf
- U24: Assembly (none) -> PLACE; MPN (none) -> TLV803EA30DBZR; Manufacturer (none) -> Texas Instruments; Procurement Source (none) -> https://www.ti.com/lit/ds/symlink/tlv803e.pdf
