File: projects/chrysler-scanner/current/24_debug-testpoints.kicad_sch (KiCad schematic)
At the start: 52 parts

Commit message: Finish Chrysler scanner CCD correction and procurement fabrication package
Parts:
- TP1, TP10, TP11, TP12, TP13, TP14, TP15, TP16, TP17, TP18, TP19, TP2, TP20, TP21, TP22, TP23, TP24, TP25, TP26, TP27, TP28, TP29, TP3, TP30, TP31, TP32, TP33, TP34, TP35, TP36, TP37, TP38, TP39, TP4, TP40, TP41, TP42, TP43, TP44, TP49, TP5, TP50, TP51, TP52, TP6, TP7, TP8, TP9: Assembly (none) -> PLACE; Procurement Source (none) -> https://www.keyelco.com/product.cfm/Micro-Miniature/5015/pr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
- TP45, TP46, TP47, TP48: Assembly (none) -> PCB_FEATURE; Procurement Source (none) -> https://www.keyelco.com/product.cfm/Micro-Miniature/5015/pr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
