File: projects/chrysler-scanner/current/08_power-5v.kicad_sch (KiCad schematic)
At the start: 17 parts, among them U2 LMR14010, U3 TLV76750DRV, U4 TLV76733DRV

Commit message: Use native ground symbols and document companion app feasibility
Other:
- note added: "All TLV767 ground terminals and exposed pads connect to GND in this checked revision."
- note added: "Native schematic and PCB ground connectivity are checked in the final validation reports."
- note removed: "REVIEW: U3 / U4 pin 5 is NC in the source; TLV767 DRV requires GND."
- note removed: "Source connectivity is preserved here. Correct this in atopile before routing."

Commit message: Fix scanner protection, ADC isolation and health watchdog
Coordinate the bounded 12 V input clamp and programming FET/capacitor ratings, add powered-off ADC isolation, and supervise the AW9523B permit with a dedicated GPIO13 health heartbeat. Preserve original placements and document all deliberate source-PDF deviations.

Validation: native ERC and full DRC/parity/refill report zero findings; strict preservation/connectivity audit and final adversarial review pass within the documented prototype bounds. Regenerate Rev C PDF, BOM, manufacturing exports, processing sites and verified portable archives. Compatible firmware and bench/mechanical qualification remain required.
Parts:
- C10, C6, C7, C8, C9: Voltage Rating (none) -> 25V
- C4: Voltage Rating (none) -> 50V
- C5: Voltage Rating (none) -> 100V

Commit message: Restore schematic polarity and visible capacitor ratings
Changed lines of the file:
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@@
 			)
 		)
-	(property "Voltage Rating" "100V" (at 0 0 0) (effects (font (size 1 1)) (hide yes))))
+	(property "Voltage Rating" "100V" (at 89.6885 56.39 0) (effects (font (size 1 1)))))
 	(symbol
 		(lib_id "power:GND")
@@
 			)
 		)
-	(property "Voltage Rating" "25V" (at 0 0 0) (effects (font (size 1 1)) (hide yes))))
+	(property "Voltage Rating" "25V" (at 241.789 94.49 0) (effects (font (size 1 1)))))
 	(symbol
 		(lib_id "power:GND")
@@
 			)
 		)
-	(property "Voltage Rating" "25V" (at 0 0 0) (effects (font (size 1 1)) (hide yes))))
+	(property "Voltage Rating" "25V" (at 340.849 94.49 0) (effects (font (size 1 1)))))
 	(symbol
 		(lib_id "ChryslerScanner:U4")
@@
 			)
 		)
-	(property "Voltage Rating" "25V" (at 0 0 0) (effects (font (size 1 1)) (hide yes))))
+	(property "Voltage Rating" "25V" (at 170.636 94.49 0) (effects (font (size 1 1)))))
 	(symbol
 		(lib_id "ChryslerScanner:R3")
@@
 			)
 		)
-	(property "Voltage Rating" "25V" (at 0 0 0) (effects (font (size 1 1)) (hide yes))))
+	(property "Voltage Rating" "25V" (at 269.696 94.49 0) (effects (font (size 1 1)))))
 	(symbol
 		(lib_id "power:GND")
@@
 			)
 		)
-	(property "Voltage Rating" "50V" (at 0 0 0) (effects (font (size 1 1)) (hide yes))))
+	(property "Voltage Rating" "50V" (at 28.3959 94.49 0) (effects (font (size 1 1)))))
 	(symbol
 		(lib_id "power:GND")
@@
 			)
 		)
-	(property "Voltage Rating" "25V" (at 0 0 0) (effects (font (size 1 1)) (hide yes))))
+	(property "Voltage Rating" "25V" (at 130.029 97.03 0) (effects (font (size 1 1)))))
 )

Commit message: Finish Chrysler scanner CCD correction and procurement fabrication package
Parts:
- C10, C6, C8: Assembly (none) -> PLACE; MPN (none) -> C3216X5R1E226M160AB; Manufacturer (none) -> TDK; Procurement Source (none) -> https://product.tdk.com/en/search/capacitor/ceramic/mlcc/in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; Selected Voltage Rating (none) -> 25V; Tolerance (none) -> 20%
- C4, C7, C9: Assembly (none) -> PLACE; MPN (none) -> CGA5L1X7R1H106K160AC; Manufacturer (none) -> TDK; Procurement Source (none) -> https://product.tdk.com/info/en/documents/chara_sheet/CGA5L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; Selected Voltage Rating (none) -> 50V; Tolerance (none) -> 10%
- C5: Assembly (none) -> PLACE; MPN (none) -> C1206C104K1RACTU; Manufacturer (none) -> KEMET; Procurement Source (none) -> https://search.kemet.com/component-documentation/download/s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; Selected Voltage Rating (none) -> 100V; Tolerance (none) -> 10%
- D4, D5, D6: Assembly (none) -> PLACE; MPN (none) -> DSK34; Manufacturer (none) -> MDD (Microdiode Electronics); Procurement Source (none) -> https://datasheet.lcsc.com/lcsc/DSK34_C41029.pdf
- L1: footprint footprints:L_7.3x7.3_H3.5 -> footprints:L_Eaton_DR74_220_R; Assembly (none) -> PLACE; MPN (none) -> DR74-220-R; Manufacturer (none) -> Eaton; Model Representation (none) -> Representative maximum overall envelope; Fab/courtyard and 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; Procurement Source (none) -> https://www.eaton.com/us/en-us/skuPage.DR74-220-R.html; Selected Height (none) -> 4.35mm max
- R1: Assembly (none) -> PLACE; MPN (none) -> CRCW0603100KFKEA; Manufacturer (none) -> Vishay; Procurement Source (none) -> https://www.vishay.com/docs/20035/dcrcwe3.pdf; Selected Power Rating (none) -> 0.1W; Tolerance (none) -> 1%
- R2: Assembly (none) -> PLACE; MPN (none) -> TNPW060368K0BEEA; Manufacturer (none) -> Vishay; Procurement Source (none) -> https://www.vishay.com/docs/28758/tnpw_e3.pdf; Selected Power Rating (none) -> 0.1W; Tolerance (none) -> 0.1%
- R3: Assembly (none) -> PLACE; MPN (none) -> TNPW060310K0BEEA; Manufacturer (none) -> Vishay; Procurement Source (none) -> https://www.vishay.com/docs/28758/tnpw_e3.pdf; Selected Power Rating (none) -> 0.1W; Tolerance (none) -> 0.1%
- U2: Assembly (none) -> PLACE; MPN (none) -> LMR14010ADDCR; Manufacturer (none) -> Texas Instruments; Procurement Source (none) -> https://www.ti.com/lit/ds/symlink/lmr14010a.pdf
- U3: Assembly (none) -> PLACE; MPN (none) -> TLV76750DRVR; Manufacturer (none) -> Texas Instruments; Procurement Source (none) -> https://www.ti.com/lit/ds/symlink/tlv767.pdf
- U4: Assembly (none) -> PLACE; MPN (none) -> TLV76733DRVR; Manufacturer (none) -> Texas Instruments; Procurement Source (none) -> https://www.ti.com/lit/ds/symlink/tlv767.pdf

Commit message: Refine programming drive, Eaton lands and mounting clearance
Parts:
- L1: footprint footprints:L_Eaton_DR74_220_R -> footprints:L_Eaton_DR74_Recommended
Changed lines of the file:
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@@
 			)
 		)
-		(property "Footprint" "footprints:L_Eaton_DR74_220_R"
+		(property "Footprint" "footprints:L_Eaton_DR74_Recommended"
 			(at 109.22 68.58 0)
 			(hide yes)
