File: projects/chrysler-scanner/current/09_power-vpp.kicad_sch (KiCad schematic)
At the start: 10 parts, among them U5 LGS6302

Commit message: Fix scanner protection, ADC isolation and health watchdog
Coordinate the bounded 12 V input clamp and programming FET/capacitor ratings, add powered-off ADC isolation, and supervise the AW9523B permit with a dedicated GPIO13 health heartbeat. Preserve original placements and document all deliberate source-PDF deviations.

Validation: native ERC and full DRC/parity/refill report zero findings; strict preservation/connectivity audit and final adversarial review pass within the documented prototype bounds. Regenerate Rev C PDF, BOM, manufacturing exports, processing sites and verified portable archives. Compatible firmware and bench/mechanical qualification remain required.
Parts:
- C13, C14, C15, C16: Voltage Rating (none) -> 50V

Commit message: Restore schematic polarity and visible capacitor ratings
Changed lines of the file:
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@@
 			)
 		)
-	(property "Voltage Rating" "50V" (at 0 0 0) (effects (font (size 1 1)) (hide yes))))
+	(property "Voltage Rating" "50V" (at 19.8641 84.33 0) (effects (font (size 1 1)))))
 	(symbol
 		(lib_id "power:GND")
@@
 			)
 		)
-	(property "Voltage Rating" "50V" (at 0 0 0) (effects (font (size 1 1)) (hide yes))))
+	(property "Voltage Rating" "50V" (at 114.789 84.33 0) (effects (font (size 1 1)))))
 	(symbol
 		(lib_id "ChryslerScanner:C16")
@@
 			)
 		)
-	(property "Voltage Rating" "50V" (at 0 0 0) (effects (font (size 1 1)) (hide yes))))
+	(property "Voltage Rating" "50V" (at 193.496 86.87 0) (effects (font (size 1 1)))))
 	(symbol
 		(lib_id "ChryslerScanner:D7")
@@
 			)
 		)
-	(property "Voltage Rating" "50V" (at 0 0 0) (effects (font (size 1 1)) (hide yes))))
+	(property "Voltage Rating" "50V" (at 165.556 84.33 0) (effects (font (size 1 1)))))
 	(symbol
 		(lib_id "power:GND")

Commit message: Finish Chrysler scanner CCD correction and procurement fabrication package
Parts:
- C13, C15, C16: Assembly (none) -> PLACE; MPN (none) -> CGA5L1X7R1H106K160AC; Manufacturer (none) -> TDK; Procurement Source (none) -> https://product.tdk.com/info/en/documents/chara_sheet/CGA5L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; Selected Voltage Rating (none) -> 50V; Tolerance (none) -> 10%
- C14: footprint footprints:C_1206_3216Metric -> footprints:C_1210_3225_TDK_22u50V; Assembly (none) -> PLACE; MPN (none) -> C3225X7R1H226M250AC; Manufacturer (none) -> TDK; Model Representation (none) -> Representative maximum overall envelope; Fab/courtyard and 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; Procurement Source (none) -> https://product.tdk.com/en/search/capacitor/ceramic/mlcc/in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; Selected Height (none) -> 2.8mm max; Selected Voltage Rating (none) -> 50V; Tolerance (none) -> 20%
- D7: Assembly (none) -> PLACE; MPN (none) -> DSK34; Manufacturer (none) -> MDD (Microdiode Electronics); Procurement Source (none) -> https://datasheet.lcsc.com/lcsc/DSK34_C41029.pdf
- L2: footprint footprints:L_7.3x7.3_H3.5 -> footprints:L_Eaton_DR74_220_R; Assembly (none) -> PLACE; MPN (none) -> DR74-220-R; Manufacturer (none) -> Eaton; Model Representation (none) -> Representative maximum overall envelope; Fab/courtyard and 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; Procurement Source (none) -> https://www.eaton.com/us/en-us/skuPage.DR74-220-R.html; Selected Height (none) -> 4.35mm max
- L3: footprint footprints:R_1206_3216Metric -> footprints:L_Bourns_SRN2012; Assembly (none) -> PLACE; MPN (none) -> SRN2012-R24M; Manufacturer (none) -> Bourns; Model Representation (none) -> Representative maximum overall envelope; Fab/courtyard and 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; Procurement Source (none) -> https://www.bourns.com/docs/product-datasheets/srn2012.pdf; Selected Height (none) -> 1.2mm max
- R8: Assembly (none) -> PLACE; MPN (none) -> TNPW0603110KBEEA; Manufacturer (none) -> Vishay; Procurement Source (none) -> https://www.vishay.com/docs/28758/tnpw_e3.pdf; Selected Power Rating (none) -> 0.1W; Tolerance (none) -> 0.1%
- R9: Assembly (none) -> PLACE; MPN (none) -> TNPW06036K80BEEA; Manufacturer (none) -> Vishay; Procurement Source (none) -> https://www.vishay.com/docs/28758/tnpw_e3.pdf; Selected Power Rating (none) -> 0.1W; Tolerance (none) -> 0.1%
- U5: Assembly (none) -> PLACE; MPN (none) -> LGS6302B5; Manufacturer (none) -> Legend-Si; Procurement Source (none) -> https://www.legend-si.com/productinfo/1318196.html
Changed lines of the file:
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@@
 			)
 		)
-		(property "Datasheet" ""
+		(property "Datasheet" "https://product.tdk.com/info/en/documents/chara_sheet/CGA5L1X7R1H106K160AC.pdf"
 			(at 27.94 81.28 0)
 			(hide yes)
@@
 			)
 		)
-	(property "Voltage Rating" "50V" (at 19.8641 84.33 0) (effects (font (size 1 1)))))
+	(property "Voltage Rating" "50V" (at 19.8641 84.33 0) (effects (font (size 1 1))))
+(property "Manufacturer" "TDK" (at 0 0 0) (effects (font (size 1 1)) (hide yes)))
+(property "MPN" "CGA5L1X7R1H106K160AC" (at 0 0 0) (effects (font (size 1 1)) (hide yes)))
+(property "Procurement Source" "https://product.tdk.com/info/en/documents/chara_sheet/CGA5L1X7R1H106K160AC.pdf" (at 0 0 0) (effects (font (size 1 1)) (hide yes)))
+(property "Assembly" "PLACE" (at 0 0 0) (effects (font (size 1 1)) (hide yes)))
+(property "Selected Voltage Rating" "50V" (at 0 0 0) (effects (font (size 1 1)) (hide yes)))
+(property "Tolerance" "10%" (at 0 0 0) (effects (font (size 1 1)) (hide yes)))
+)
 	(symbol
 		(lib_id "power:GND")
@@
 			)
 		)
-		(property "Footprint" "footprints:C_1206_3216Metric"
+		(property "Footprint" "footprints:C_1210_3225_TDK_22u50V"
 			(at 106.68 81.28 0)
 			(hide yes)
@@
 			)
 		)
-		(property "Datasheet" ""
+		(property "Datasheet" "https://product.tdk.com/en/search/capacitor/ceramic/mlcc/info?part_no=C3225X7R1H226M250AC"
 			(at 106.68 81.28 0)
 			(hide yes)
@@
 			)
 		)
-	(property "Voltage Rating" "50V" (at 114.789 84.33 0) (effects (font (size 1 1)))))
+	(property "Voltage Rating" "50V" (at 114.789 84.33 0) (effects (font (size 1 1))))
+(property "Manufacturer" "TDK" (at 0 0 0) (effects (font (size 1 1)) (hide yes)))
+(property "MPN" "C3225X7R1H226M250AC" (at 0 0 0) (effects (font (size 1 1)) (hide yes)))
+(property "Procurement Source" "https://product.tdk.com/en/search/capacitor/ceramic/mlcc/info?part_no=C3225X7R1H226M250AC" (at 0 0 0) (effects (font (size 1 1)) (hide yes)))
+(property "Assembly" "PLACE" (at 0 0 0) (effects (font (size 1 1)) (hide yes)))
+(property "Selected Voltage Rating" "50V" (at 0 0 0) (effects (font (size 1 1)) (hide yes)))
+(property "Tolerance" "20%" (at 0 0 0) (effects (font (size 1 1)) (hide yes)))
+(property "Selected Height" "2.8mm max" (at 0 0 0) (effects (font (size 1 1)) (hide yes)))
+(property "Model Representation" "Representative maximum overall envelope; Fab/courtyard and selected dimensions govern fit." (at 0 0 0) (effects (font (size 1 1)) (hide yes)))
+)
 	(symbol
 		(lib_id "ChryslerScanner:C16")
@@
 			)
 		)
-		(property "Datasheet" ""
+		(property "Datasheet" "https://product.tdk.com/info/en/documents/chara_sheet/CGA5L1X7R1H106K160AC.pdf"
 			(at 185.42 83.82 0)
 			(hide yes)
@@
 			)
 		)
-	(property "Voltage Rating" "50V" (at 193.496 86.87 0) (effects (font (size 1 1)))))
+	(property "Voltage Rating" "50V" (at 193.496 86.87 0) (effects (font (size 1 1))))
+(property "Manufacturer" "TDK" (at 0 0 0) (effects (font (size 1 1)) (hide yes)))
+(property "MPN" "CGA5L1X7R1H106K160AC" (at 0 0 0) (effects (font (size 1 1)) (hide yes)))
+(property "Procurement Source" "https://product.tdk.com/info/en/documents/chara_sheet/CGA5L1X7R1H106K160AC.pdf" (at 0 0 0) (effects (font (size 1 1)) (hide yes)))
+(property "Assembly" "PLACE" (at 0 0 0) (effects (font (size 1 1)) (hide yes)))
+(property "Selected Voltage Rating" "50V" (at 0 0 0) (effects (font (size 1 1)) (hide yes)))
+(property "Tolerance" "10%" (at 0 0 0) (effects (font (size 1 1)) (hide yes)))
+)
 	(symbol
 		(lib_id "ChryslerScanner:D7")
@@
 			)
 		)
-		(property "Datasheet" ""
+		(property "Datasheet" "https://datasheet.lcsc.com/lcsc/DSK34_C41029.pdf"
 			(at 93.98 50.8 0)
 			(hide yes)
@@
 			)
 		)
-	)
+(property "Manufacturer" "MDD (Microdiode Electronics)" (at 0 0 0) (effects (font (size 1 1)) (hide yes)))
+(property "MPN" "DSK34" (at 0 0 0) (effects (font (size 1 1)) (hide yes)))
+(property "Procurement Source" "https://datasheet.lcsc.com/lcsc/DSK34_C41029.pdf" (at 0 0 0) (effects (font (size 1 1)) (hide yes)))
+(property "Assembly" "PLACE" (at 0 0 0) (effects (font (size 1 1)) (hide yes)))
+)
 	(symbol
 		(lib_id "ChryslerScanner:L3")
@@
 			)
 		)
-		(property "Footprint" "footprints:R_1206_3216Metric"
+		(property "Footprint" "footprints:L_Bourns_SRN2012"
 			(at 144.78 50.8 0)
 			(hide yes)
@@
 			)
 		)
-		(property "Datasheet" ""
+		(property "Datasheet" "https://www.bourns.com/docs/product-datasheets/srn2012.pdf"
 			(at 144.78 50.8 0)
 			(hide yes)
@@
 			)
 		)
-	)
+(property "Manufacturer" "Bourns" (at 0 0 0) (effects (font (size 1 1)) (hide yes)))
+(property "MPN" "SRN2012-R24M" (at 0 0 0) (effects (font (size 1 1)) (hide yes)))
+(property "Procurement Source" "https://www.bourns.com/docs/product-datasheets/srn2012.pdf" (at 0 0 0) (effects (font (size 1 1)) (hide yes)))
+(property "Assembly" "PLACE" (at 0 0 0) (effects (font (size 1 1)) (hide yes)))
+(property "Selected Height" "1.2mm max" (at 0 0 0) (effects (font (size 1 1)) (hide yes)))
+(property "Model Representation" "Representative maximum overall envelope; Fab/courtyard and selected dimensions govern fit." (at 0 0 0) (effects (font (size 1 1)) (hide yes)))
+)
 	(symbol
 		(lib_id "power:GND")
@@
 			)
 		)
-		(property "Datasheet" ""
+		(property "Datasheet" "https://www.vishay.com/docs/28758/tnpw_e3.pdf"
 			(at 132.08 91.44 0)
 			(hide yes)
@@
 			)
 		)
-	)
+(property "Manufacturer" "Vishay" (at 0 0 0) (effects (font (size 1 1)) (hide yes)))
+(property "MPN" "TNPW06036K80BEEA" (at 0 0 0) (effects (font (size 1 1)) (hide yes)))
+(property "Procurement Source" "https://www.vishay.com/docs/28758/tnpw_e3.pdf" (at 0 0 0) (effects (font (size 1 1)) (hide yes)))
+(property "Assembly" "PLACE" (at 0 0 0) (effects (font (size 1 1)) (hide yes)))
+(property "Tolerance" "0.1%" (at 0 0 0) (effects (font (size 1 1)) (hide yes)))
+(property "Selected Power Rating" "0.1W" (at 0 0 0) (effects (font (size 1 1)) (hide yes)))
+)
 	(symbol
 		(lib_id "ChryslerScanner:R8")
@@
 			)
 		)
-		(property "Datasheet" ""
+		(property "Datasheet" "https://www.vishay.com/docs/28758/tnpw_e3.pdf"
 			(at 132.08 71.12 0)
 			(hide yes)
@@
 			)
 		)
-	)
+(property "Manufacturer" "Vishay" (at 0 0 0) (effects (font (size 1 1)) (hide yes)))
+(property "MPN" "TNPW0603110KBEEA" (at 0 0 0) (effects (font (size 1 1)) (hide yes)))
+(property "Procurement Source" "https://www.vishay.com/docs/28758/tnpw_e3.pdf" (at 0 0 0) (effects (font (size 1 1)) (hide yes)))
+(property "Assembly" "PLACE" (at 0 0 0) (effects (font (size 1 1)) (hide yes)))
+(property "Tolerance" "0.1%" (at 0 0 0) (effects (font (size 1 1)) (hide yes)))
+(property "Selected Power Rating" "0.1W" (at 0 0 0) (effects (font (size 1 1)) (hide yes)))
+)
 	(symbol
 		(lib_id "power:GND")
@@
 			)
 		)
-		(property "Datasheet" ""
+		(property "Datasheet" "https://www.legend-si.com/productinfo/1318196.html"
 			(at 60.96 81.28 0)
 			(hide yes)
@@
 			)
 		)
-	)
+(property "Manufacturer" "Legend-Si" (at 0 0 0) (effects (font (size 1 1)) (hide yes)))
+(property "MPN" "LGS6302B5" (at 0 0 0) (effects (font (size 1 1)) (hide yes)))
+(property "Procurement Source" "https://www.legend-si.com/productinfo/1318196.html" (at 0 0 0) (effects (font (size 1 1)) (hide yes)))
+(property "Assembly" "PLACE" (at 0 0 0) (effects (font (size 1 1)) (hide yes)))
+)
 	(symbol
 		(lib_id "ChryslerScanner:L2")
@@
 			)
 		)
-		(property "Footprint" "footprints:L_7.3x7.3_H3.5"
+		(property "Footprint" "footprints:L_Eaton_DR74_220_R"
 			(at 60.96 50.8 0)
 			(hide yes)
@@
 			)
 		)
-		(property "Datasheet" ""
+		(property "Datasheet" "https://www.eaton.com/us/en-us/skuPage.DR74-220-R.html"
 			(at 60.96 50.8 0)
 			(hide yes)
@@
 			)
 		)
-	)
+(property "Manufacturer" "Eaton" (at 0 0 0) (effects (font (size 1 1)) (hide yes)))
+(property "MPN" "DR74-220-R" (at 0 0 0) (effects (font (size 1 1)) (hide yes)))
+(property "Procurement Source" "https://www.eaton.com/us/en-us/skuPage.DR74-220-R.html" (at 0 0 0) (effects (font (size 1 1)) (hide yes)))
+(property "Assembly" "PLACE" (at 0 0 0) (effects (font (size 1 1)) (hide yes)))
+(property "Selected Height" "4.35mm max" (at 0 0 0) (effects (font (size 1 1)) (hide yes)))
+(property "Model Representation" "Representative maximum overall envelope; Fab/courtyard and selected dimensions govern fit." (at 0 0 0) (effects (font (size 1 1)) (hide yes)))
+)
 	(symbol
 		(lib_id "ChryslerScanner:C15")
@@
 			)
 		)
-		(property "Datasheet" ""
+		(property "Datasheet" "https://product.tdk.com/info/en/documents/chara_sheet/CGA5L1X7R1H106K160AC.pdf"
 			(at 157.48 81.28 0)
 			(hide yes)
@@
 			)
 		)
-	(property "Voltage Rating" "50V" (at 165.556 84.33 0) (effects (font (size 1 1)))))
+	(property "Voltage Rating" "50V" (at 165.556 84.33 0) (effects (font (size 1 1))))
+(property "Manufacturer" "TDK" (at 0 0 0) (effects (font (size 1 1)) (hide yes)))
+(property "MPN" "CGA5L1X7R1H106K160AC" (at 0 0 0) (effects (font (size 1 1)) (hide yes)))
+(property "Procurement Source" "https://product.tdk.com/info/en/documents/chara_sheet/CGA5L1X7R1H106K160AC.pdf" (at 0 0 0) (effects (font (size 1 1)) (hide yes)))
+(property "Assembly" "PLACE" (at 0 0 0) (effects (font (size 1 1)) (hide yes)))
+(property "Selected Voltage Rating" "50V" (at 0 0 0) (effects (font (size 1 1)) (hide yes)))
+(property "Tolerance" "10%" (at 0 0 0) (effects (font (size 1 1)) (hide yes)))
+)
 	(symbol
 		(lib_id "power:GND")

Commit message: Refine programming drive, Eaton lands and mounting clearance
Parts:
- L2: footprint footprints:L_Eaton_DR74_220_R -> footprints:L_Eaton_DR74_Recommended
Changed lines of the file:
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@@
 			)
 		)
-		(property "Footprint" "footprints:L_Eaton_DR74_220_R"
+		(property "Footprint" "footprints:L_Eaton_DR74_Recommended"
 			(at 60.96 50.8 0)
 			(hide yes)
