File: projects/chrysler-scanner/current/10_power-vbb.kicad_sch (KiCad schematic)
At the start: 10 parts, among them U6 LMR14010

Commit message: Fix scanner protection, ADC isolation and health watchdog
Coordinate the bounded 12 V input clamp and programming FET/capacitor ratings, add powered-off ADC isolation, and supervise the AW9523B permit with a dedicated GPIO13 health heartbeat. Preserve original placements and document all deliberate source-PDF deviations.

Validation: native ERC and full DRC/parity/refill report zero findings; strict preservation/connectivity audit and final adversarial review pass within the documented prototype bounds. Regenerate Rev C PDF, BOM, manufacturing exports, processing sites and verified portable archives. Compatible firmware and bench/mechanical qualification remain required.
Parts:
- C17: Voltage Rating (none) -> 100V
- C18, C19: Voltage Rating (none) -> 25V

Commit message: Restore schematic polarity and visible capacitor ratings
Changed lines of the file:
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@@
 			)
 		)
-	(property "Voltage Rating" "100V" (at 0 0 0) (effects (font (size 1 1)) (hide yes))))
+	(property "Voltage Rating" "100V" (at 87.1485 48.77 0) (effects (font (size 1 1)))))
 	(symbol
 		(lib_id "ChryslerScanner:R10")
@@
 			)
 		)
-	(property "Voltage Rating" "25V" (at 0 0 0) (effects (font (size 1 1)) (hide yes))))
+	(property "Voltage Rating" "25V" (at 127.489 86.87 0) (effects (font (size 1 1)))))
 	(symbol
 		(lib_id "ChryslerScanner:L5")
@@
 			)
 		)
-	(property "Voltage Rating" "25V" (at 0 0 0) (effects (font (size 1 1)) (hide yes))))
+	(property "Voltage Rating" "25V" (at 178.256 86.87 0) (effects (font (size 1 1)))))
 	(symbol
 		(lib_id "ChryslerScanner:R12")

Commit message: Finish Chrysler scanner CCD correction and procurement fabrication package
Parts:
- C17: Assembly (none) -> PLACE; MPN (none) -> C1206C104K1RACTU; Manufacturer (none) -> KEMET; Procurement Source (none) -> https://search.kemet.com/component-documentation/download/s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; Selected Voltage Rating (none) -> 100V; Tolerance (none) -> 10%
- C18: Assembly (none) -> PLACE; MPN (none) -> C3216X5R1E226M160AB; Manufacturer (none) -> TDK; Procurement Source (none) -> https://product.tdk.com/en/search/capacitor/ceramic/mlcc/in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; Selected Voltage Rating (none) -> 25V; Tolerance (none) -> 20%
- C19: Assembly (none) -> PLACE; MPN (none) -> CGA5L1X7R1H106K160AC; Manufacturer (none) -> TDK; Procurement Source (none) -> https://product.tdk.com/info/en/documents/chara_sheet/CGA5L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; Selected Voltage Rating (none) -> 50V; Tolerance (none) -> 10%
- D8: Assembly (none) -> PLACE; MPN (none) -> DSK34; Manufacturer (none) -> MDD (Microdiode Electronics); Procurement Source (none) -> https://datasheet.lcsc.com/lcsc/DSK34_C41029.pdf
- L4: footprint footprints:L_7.3x7.3_H3.5 -> footprints:L_Eaton_DR74_220_R; Assembly (none) -> PLACE; MPN (none) -> DR74-220-R; Manufacturer (none) -> Eaton; Model Representation (none) -> Representative maximum overall envelope; Fab/courtyard and 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; Procurement Source (none) -> https://www.eaton.com/us/en-us/skuPage.DR74-220-R.html; Selected Height (none) -> 4.35mm max
- L5: footprint footprints:R_1206_3216Metric -> footprints:L_Bourns_SRN2012; Assembly (none) -> PLACE; MPN (none) -> SRN2012-R47M; Manufacturer (none) -> Bourns; Model Representation (none) -> Representative maximum overall envelope; Fab/courtyard and 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; Procurement Source (none) -> https://www.bourns.com/docs/product-datasheets/srn2012.pdf; Selected Height (none) -> 1.2mm max
- R10: Assembly (none) -> PLACE; MPN (none) -> CRCW0603100KFKEA; Manufacturer (none) -> Vishay; Procurement Source (none) -> https://www.vishay.com/docs/20035/dcrcwe3.pdf; Selected Power Rating (none) -> 0.1W; Tolerance (none) -> 1%
- R11: Assembly (none) -> PLACE; MPN (none) -> TNPW0603158KBEEA; Manufacturer (none) -> Vishay; Procurement Source (none) -> https://www.vishay.com/docs/28758/tnpw_e3.pdf; Selected Power Rating (none) -> 0.1W; Tolerance (none) -> 0.1%
- R12: Assembly (none) -> PLACE; MPN (none) -> TNPW060310K0BEEA; Manufacturer (none) -> Vishay; Procurement Source (none) -> https://www.vishay.com/docs/28758/tnpw_e3.pdf; Selected Power Rating (none) -> 0.1W; Tolerance (none) -> 0.1%
- U6: Assembly (none) -> PLACE; MPN (none) -> LMR14010ADDCR; Manufacturer (none) -> Texas Instruments; Procurement Source (none) -> https://www.ti.com/lit/ds/symlink/lmr14010a.pdf
Changed lines of the file:
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@@
 			)
 		)
-		(property "Datasheet" ""
+		(property "Datasheet" "https://search.kemet.com/component-documentation/download/specsheet/C1206C104K1RACTU"
 			(at 81.28 50.8 0)
 			(hide yes)
@@
 			)
 		)
-	(property "Voltage Rating" "100V" (at 87.1485 48.77 0) (effects (font (size 1 1)))))
+	(property "Voltage Rating" "100V" (at 87.1485 48.77 0) (effects (font (size 1 1))))
+(property "Manufacturer" "KEMET" (at 0 0 0) (effects (font (size 1 1)) (hide yes)))
+(property "MPN" "C1206C104K1RACTU" (at 0 0 0) (effects (font (size 1 1)) (hide yes)))
+(property "Procurement Source" "https://search.kemet.com/component-documentation/download/specsheet/C1206C104K1RACTU" (at 0 0 0) (effects (font (size 1 1)) (hide yes)))
+(property "Assembly" "PLACE" (at 0 0 0) (effects (font (size 1 1)) (hide yes)))
+(property "Selected Voltage Rating" "100V" (at 0 0 0) (effects (font (size 1 1)) (hide yes)))
+(property "Tolerance" "10%" (at 0 0 0) (effects (font (size 1 1)) (hide yes)))
+)
 	(symbol
 		(lib_id "ChryslerScanner:R10")
@@
 			)
 		)
-		(property "Datasheet" ""
+		(property "Datasheet" "https://www.vishay.com/docs/20035/dcrcwe3.pdf"
 			(at 30.48 60.96 0)
 			(hide yes)
@@
 			)
 		)
-	)
+(property "Manufacturer" "Vishay" (at 0 0 0) (effects (font (size 1 1)) (hide yes)))
+(property "MPN" "CRCW0603100KFKEA" (at 0 0 0) (effects (font (size 1 1)) (hide yes)))
+(property "Procurement Source" "https://www.vishay.com/docs/20035/dcrcwe3.pdf" (at 0 0 0) (effects (font (size 1 1)) (hide yes)))
+(property "Assembly" "PLACE" (at 0 0 0) (effects (font (size 1 1)) (hide yes)))
+(property "Tolerance" "1%" (at 0 0 0) (effects (font (size 1 1)) (hide yes)))
+(property "Selected Power Rating" "0.1W" (at 0 0 0) (effects (font (size 1 1)) (hide yes)))
+)
 	(symbol
 		(lib_id "ChryslerScanner:D8")
@@
 			)
 		)
-		(property "Datasheet" ""
+		(property "Datasheet" "https://datasheet.lcsc.com/lcsc/DSK34_C41029.pdf"
 			(at 93.98 83.82 0)
 			(hide yes)
@@
 			)
 		)
-	)
+(property "Manufacturer" "MDD (Microdiode Electronics)" (at 0 0 0) (effects (font (size 1 1)) (hide yes)))
+(property "MPN" "DSK34" (at 0 0 0) (effects (font (size 1 1)) (hide yes)))
+(property "Procurement Source" "https://datasheet.lcsc.com/lcsc/DSK34_C41029.pdf" (at 0 0 0) (effects (font (size 1 1)) (hide yes)))
+(property "Assembly" "PLACE" (at 0 0 0) (effects (font (size 1 1)) (hide yes)))
+)
 	(symbol
 		(lib_id "ChryslerScanner:L4")
@@
 			)
 		)
-		(property "Footprint" "footprints:L_7.3x7.3_H3.5"
+		(property "Footprint" "footprints:L_Eaton_DR74_220_R"
 			(at 106.68 60.96 0)
 			(hide yes)
@@
 			)
 		)
-		(property "Datasheet" ""
+		(property "Datasheet" "https://www.eaton.com/us/en-us/skuPage.DR74-220-R.html"
 			(at 106.68 60.96 0)
 			(hide yes)
@@
 			)
 		)
-	)
+(property "Manufacturer" "Eaton" (at 0 0 0) (effects (font (size 1 1)) (hide yes)))
+(property "MPN" "DR74-220-R" (at 0 0 0) (effects (font (size 1 1)) (hide yes)))
+(property "Procurement Source" "https://www.eaton.com/us/en-us/skuPage.DR74-220-R.html" (at 0 0 0) (effects (font (size 1 1)) (hide yes)))
+(property "Assembly" "PLACE" (at 0 0 0) (effects (font (size 1 1)) (hide yes)))
+(property "Selected Height" "4.35mm max" (at 0 0 0) (effects (font (size 1 1)) (hide yes)))
+(property "Model Representation" "Representative maximum overall envelope; Fab/courtyard and selected dimensions govern fit." (at 0 0 0) (effects (font (size 1 1)) (hide yes)))
+)
 	(symbol
 		(lib_id "ChryslerScanner:C18")
@@
 			)
 		)
-		(property "Datasheet" ""
+		(property "Datasheet" "https://product.tdk.com/en/search/capacitor/ceramic/mlcc/info?part_no=C3216X5R1E226M160AB"
 			(at 119.38 83.82 0)
 			(hide yes)
@@
 			)
 		)
-	(property "Voltage Rating" "25V" (at 127.489 86.87 0) (effects (font (size 1 1)))))
+	(property "Voltage Rating" "25V" (at 127.489 86.87 0) (effects (font (size 1 1))))
+(property "Manufacturer" "TDK" (at 0 0 0) (effects (font (size 1 1)) (hide yes)))
+(property "MPN" "C3216X5R1E226M160AB" (at 0 0 0) (effects (font (size 1 1)) (hide yes)))
+(property "Procurement Source" "https://product.tdk.com/en/search/capacitor/ceramic/mlcc/info?part_no=C3216X5R1E226M160AB" (at 0 0 0) (effects (font (size 1 1)) (hide yes)))
+(property "Assembly" "PLACE" (at 0 0 0) (effects (font (size 1 1)) (hide yes)))
+(property "Selected Voltage Rating" "25V" (at 0 0 0) (effects (font (size 1 1)) (hide yes)))
+(property "Tolerance" "20%" (at 0 0 0) (effects (font (size 1 1)) (hide yes)))
+)
 	(symbol
 		(lib_id "ChryslerScanner:L5")
@@
 			)
 		)
-		(property "Footprint" "footprints:R_1206_3216Metric"
+		(property "Footprint" "footprints:L_Bourns_SRN2012"
 			(at 157.48 60.96 0)
 			(hide yes)
@@
 			)
 		)
-		(property "Datasheet" ""
+		(property "Datasheet" "https://www.bourns.com/docs/product-datasheets/srn2012.pdf"
 			(at 157.48 60.96 0)
 			(hide yes)
@@
 			)
 		)
-	)
+(property "Manufacturer" "Bourns" (at 0 0 0) (effects (font (size 1 1)) (hide yes)))
+(property "MPN" "SRN2012-R47M" (at 0 0 0) (effects (font (size 1 1)) (hide yes)))
+(property "Procurement Source" "https://www.bourns.com/docs/product-datasheets/srn2012.pdf" (at 0 0 0) (effects (font (size 1 1)) (hide yes)))
+(property "Assembly" "PLACE" (at 0 0 0) (effects (font (size 1 1)) (hide yes)))
+(property "Selected Height" "1.2mm max" (at 0 0 0) (effects (font (size 1 1)) (hide yes)))
+(property "Model Representation" "Representative maximum overall envelope; Fab/courtyard and selected dimensions govern fit." (at 0 0 0) (effects (font (size 1 1)) (hide yes)))
+)
 	(symbol
 		(lib_id "ChryslerScanner:C19")
@@
 			)
 		)
-		(property "Datasheet" ""
+		(property "Datasheet" "https://product.tdk.com/info/en/documents/chara_sheet/CGA5L1X7R1H106K160AC.pdf"
 			(at 170.18 83.82 0)
 			(hide yes)
@@
 			)
 		)
-	(property "Voltage Rating" "25V" (at 178.256 86.87 0) (effects (font (size 1 1)))))
+	(property "Voltage Rating" "25V" (at 178.256 86.87 0) (effects (font (size 1 1))))
+(property "Manufacturer" "TDK" (at 0 0 0) (effects (font (size 1 1)) (hide yes)))
+(property "MPN" "CGA5L1X7R1H106K160AC" (at 0 0 0) (effects (font (size 1 1)) (hide yes)))
+(property "Procurement Source" "https://product.tdk.com/info/en/documents/chara_sheet/CGA5L1X7R1H106K160AC.pdf" (at 0 0 0) (effects (font (size 1 1)) (hide yes)))
+(property "Assembly" "PLACE" (at 0 0 0) (effects (font (size 1 1)) (hide yes)))
+(property "Selected Voltage Rating" "50V" (at 0 0 0) (effects (font (size 1 1)) (hide yes)))
+(property "Tolerance" "10%" (at 0 0 0) (effects (font (size 1 1)) (hide yes)))
+)
 	(symbol
 		(lib_id "ChryslerScanner:R12")
@@
 			)
 		)
-		(property "Datasheet" ""
+		(property "Datasheet" "https://www.vishay.com/docs/28758/tnpw_e3.pdf"
 			(at 144.78 93.98 0)
 			(hide yes)
@@
 			)
 		)
-	)
+(property "Manufacturer" "Vishay" (at 0 0 0) (effects (font (size 1 1)) (hide yes)))
+(property "MPN" "TNPW060310K0BEEA" (at 0 0 0) (effects (font (size 1 1)) (hide yes)))
+(property "Procurement Source" "https://www.vishay.com/docs/28758/tnpw_e3.pdf" (at 0 0 0) (effects (font (size 1 1)) (hide yes)))
+(property "Assembly" "PLACE" (at 0 0 0) (effects (font (size 1 1)) (hide yes)))
+(property "Tolerance" "0.1%" (at 0 0 0) (effects (font (size 1 1)) (hide yes)))
+(property "Selected Power Rating" "0.1W" (at 0 0 0) (effects (font (size 1 1)) (hide yes)))
+)
 	(symbol
 		(lib_id "ChryslerScanner:R11")
@@
 			)
 		)
-		(property "Datasheet" ""
+		(property "Datasheet" "https://www.vishay.com/docs/28758/tnpw_e3.pdf"
 			(at 144.78 73.66 0)
 			(hide yes)
@@
 			)
 		)
-	)
+(property "Manufacturer" "Vishay" (at 0 0 0) (effects (font (size 1 1)) (hide yes)))
+(property "MPN" "TNPW0603158KBEEA" (at 0 0 0) (effects (font (size 1 1)) (hide yes)))
+(property "Procurement Source" "https://www.vishay.com/docs/28758/tnpw_e3.pdf" (at 0 0 0) (effects (font (size 1 1)) (hide yes)))
+(property "Assembly" "PLACE" (at 0 0 0) (effects (font (size 1 1)) (hide yes)))
+(property "Tolerance" "0.1%" (at 0 0 0) (effects (font (size 1 1)) (hide yes)))
+(property "Selected Power Rating" "0.1W" (at 0 0 0) (effects (font (size 1 1)) (hide yes)))
+)
 	(symbol
 		(lib_id "power:GND")
@@
 			)
 		)
-		(property "Datasheet" ""
+		(property "Datasheet" "https://www.ti.com/lit/ds/symlink/lmr14010a.pdf"
 			(at 58.42 60.96 0)
 			(hide yes)
@@
 			)
 		)
-	)
+(property "Manufacturer" "Texas Instruments" (at 0 0 0) (effects (font (size 1 1)) (hide yes)))
+(property "MPN" "LMR14010ADDCR" (at 0 0 0) (effects (font (size 1 1)) (hide yes)))
+(property "Procurement Source" "https://www.ti.com/lit/ds/symlink/lmr14010a.pdf" (at 0 0 0) (effects (font (size 1 1)) (hide yes)))
+(property "Assembly" "PLACE" (at 0 0 0) (effects (font (size 1 1)) (hide yes)))
+)
 	(symbol
 		(lib_id "power:GND")

Commit message: Refine programming drive, Eaton lands and mounting clearance
Parts:
- L4: footprint footprints:L_Eaton_DR74_220_R -> footprints:L_Eaton_DR74_Recommended
Changed lines of the file:
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@@
 			)
 		)
-		(property "Footprint" "footprints:L_Eaton_DR74_220_R"
+		(property "Footprint" "footprints:L_Eaton_DR74_Recommended"
 			(at 106.68 60.96 0)
 			(hide yes)
