File: projects/chrysler-scanner/current/12_program-6.kicad_sch (KiCad schematic)
At the start: 9 parts, among them Q12 DMG6601LVT-7, Q8 DMC3071LVT-7

Commit message: Refine programming drive, Eaton lands and mounting clearance
Parts:
- added R124: 8.2k 1%, footprints:R_0603_1608Metric, symbol ChryslerScanner:R124
- Q8: value DMC3071LVT-7 -> DMG6601LVT-7; MPN DMC3071LVT-7 -> DMG6601LVT-7; Procurement Source https://www.diodes.com/datasheet/download/DMC3071LVT.pdf -> https://www.diodes.com/datasheet/download/DMG6601LVT.pdf
Connections:
- net N_R56_2: now also R124.2; no longer Q8.6
- new net N_R124_1: Q8.6, R124.1
Other:
- note added: "VBB gate divider: 4.7k / 8.2k limits |Vgs| to 10.34V at the bounded 28V peak. AW9523 P0 must be configured push-pull; startup/default controls stay low."
Changed lines of the file:
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@@
 	(wire
 		(pts
-			(xy 50.8 73.66) (xy 66.04 73.66)
+			(xy 121.92 99.06) (xy 121.92 104.14)
 		)
 		(stroke
@@
 	(wire
 		(pts
-			(xy 121.92 99.06) (xy 121.92 104.14)
+			(xy 50.8 73.66) (xy 50.8 78.74)
 		)
 		(stroke
@@
 	(wire
 		(pts
-			(xy 50.8 73.66) (xy 50.8 78.74)
+			(xy 50.8 99.06) (xy 50.8 113.03)
 		)
 		(stroke
@@
 	(wire
 		(pts
-			(xy 50.8 99.06) (xy 50.8 113.03)
+			(xy 121.92 124.46) (xy 121.92 128.27)
 		)
 		(stroke
@@
 	(wire
 		(pts
-			(xy 121.92 124.46) (xy 121.92 128.27)
+			(xy 167.64 48.26) (xy 167.64 63.5)
 		)
 		(stroke
@@
 	(wire
 		(pts
-			(xy 167.64 48.26) (xy 167.64 63.5)
+			(xy 78.74 48.26) (xy 78.74 63.5)
 		)
 		(stroke
@@
 	(wire
 		(pts
-			(xy 78.74 48.26) (xy 78.74 63.5)
+			(xy 167.64 43.18) (xy 167.64 48.26)
 		)
 		(stroke
@@
 	(wire
 		(pts
-			(xy 167.64 43.18) (xy 167.64 48.26)
+			(xy 33.02 83.82) (xy 33.02 88.9)
 		)
 		(stroke
@@
 	(wire
 		(pts
-			(xy 50.8 68.58) (xy 50.8 73.66)
+			(xy 139.7 68.58) (xy 139.7 73.66)
 		)
 		(stroke
@@
 	(wire
 		(pts
-			(xy 33.02 83.82) (xy 33.02 88.9)
+			(xy 121.92 104.14) (xy 121.92 109.22)
 		)
 		(stroke
@@
 	(wire
 		(pts
-			(xy 139.7 68.58) (xy 139.7 73.66)
+			(xy 139.7 114.3) (xy 139.7 128.27)
 		)
 		(stroke
@@
 	(wire
 		(pts
-			(xy 121.92 104.14) (xy 121.92 109.22)
+			(xy 33.02 109.22) (xy 33.02 113.03)
 		)
 		(stroke
@@
 	(wire
 		(pts
-			(xy 139.7 114.3) (xy 139.7 128.27)
+			(xy 33.02 88.9) (xy 33.02 93.98)
 		)
 		(stroke
@@
 	(wire
 		(pts
-			(xy 33.02 109.22) (xy 33.02 113.03)
+			(xy 121.92 104.14) (xy 127 104.14)
 		)
 		(stroke
@@
 	(wire
 		(pts
-			(xy 33.02 88.9) (xy 33.02 93.98)
+			(xy 50.8 53.34) (xy 50.8 48.26)
 		)
 		(stroke
@@
 		)
 	)
-	(wire
-		(pts
-			(xy 121.92 104.14) (xy 127 104.14)
-		)
-		(stroke
-			(width 0)
-			(type default)
-		)
-	)
-	(wire
-		(pts
-			(xy 50.8 53.34) (xy 50.8 48.26)
-		)
-		(stroke
-			(width 0)
-			(type default)
-		)
-	)
-	(global_label "N_R56_2"
+	(global_label "N_R124_1"
 		(shape input)
 		(at 50.8 78.74 0)
@@
 			)
 		)
-		(property "Value" "DMC3071LVT-7"
+		(property "Value" "DMG6601LVT-7"
 			(at 60.7506 89.85 0)
 			(show_name no)
@@
 			)
 		)
-		(property "Datasheet" "https://www.diodes.com/datasheet/download/DMC3071LVT.pdf"
+		(property "Datasheet" "https://www.diodes.com/datasheet/download/DMG6601LVT.pdf"
 			(at 49.022 88.9 0)
 			(hide yes)
@@
 		)
 (property "Manufacturer" "Diodes Incorporated" (at 0 0 0) (effects (font (size 1 1)) (hide yes)))
-(property "MPN" "DMC3071LVT-7" (at 0 0 0) (effects (font (size 1 1)) (hide yes)))
-(property "Procurement Source" "https://www.diodes.com/datasheet/download/DMC3071LVT.pdf" (at 0 0 0) (effects (font (size 1 1)) (hide yes)))
+(property "MPN" "DMG6601LVT-7" (at 0 0 0) (effects (font (size 1 1)) (hide yes)))
+(property "Procurement Source" "https://www.diodes.com/datasheet/download/DMG6601LVT.pdf" (at 0 0 0) (effects (font (size 1 1)) (hide yes)))
 (property "Assembly" "PLACE" (at 0 0 0) (effects (font (size 1 1)) (hide yes)))
 )
@@
 			)
 		)
-		(property "Value" "DMC3071LVT-7"
+		(property "Value" "DMG6601LVT-7"
 			(at 88.6906 74.61 0)
 			(show_name no)
@@
 			)
 		)
-		(property "Datasheet" "https://www.diodes.com/datasheet/download/DMC3071LVT.pdf"
+		(property "Datasheet" "https://www.diodes.com/datasheet/download/DMG6601LVT.pdf"
 			(at 76.962 73.66 0)
 			(hide yes)
@@
 		)
 (property "Manufacturer" "Diodes Incorporated" (at 0 0 0) (effects (font (size 1 1)) (hide yes)))
-(property "MPN" "DMC3071LVT-7" (at 0 0 0) (effects (font (size 1 1)) (hide yes)))
-(property "Procurement Source" "https://www.diodes.com/datasheet/download/DMC3071LVT.pdf" (at 0 0 0) (effects (font (size 1 1)) (hide yes)))
+(property "MPN" "DMG6601LVT-7" (at 0 0 0) (effects (font (size 1 1)) (hide yes)))
+(property "Procurement Source" "https://www.diodes.com/datasheet/download/DMG6601LVT.pdf" (at 0 0 0) (effects (font (size 1 1)) (hide yes)))
 (property "Assembly" "PLACE" (at 0 0 0) (effects (font (size 1 1)) (hide yes)))
 )
@@
 (property "Assembly" "PLACE" (at 0 0 0) (effects (font (size 1 1)) (hide yes)))
 )
-)
+(symbol (lib_id "ChryslerScanner:R124") (at 58.42 73.66 0) (unit 1) (in_bom yes) (on_board yes) (dnp no)(property "Reference" "R124" (at 58.42 70.6 0) (effects (font (size 1 1))))(property "Value" "8.2k 1%" (at 58.42 76.7 0) (effects (font (size 1 1))))(property "Footprint" "footprints:R_0603_1608Metric" (at 58.42 73.66 0) (effects (font (size 1 1))(hide yes)))(property "Datasheet" "https://www.vishay.com/docs/20035/dcrcwe3.pdf" (at 58.42 73.66 0) (effects (font (size 1 1))(hide yes)))(property "Manufacturer" "Vishay" (at 58.42 73.66 0) (effects (font (size 1 1))(hide yes)))(property "MPN" "CRCW06038K20FKEA" (at 58.42 73.66 0) (effects (font (size 1 1))(hide yes)))(property "Procurement Source" "https://www.vishay.com/docs/20035/dcrcwe3.pdf" (at 58.42 73.66 0) (effects (font (size 1 1))(hide yes)))(property "Assembly" "PLACE" (at 58.42 73.66 0) (effects (font (size 1 1))(hide yes)))(property "Tolerance" "1%" (at 58.42 73.66 0) (effects (font (size 1 1))(hide yes)))(property "Selected Power Rating" "0.1W" (at 58.42 73.66 0) (effects (font (size 1 1))(hide yes)))(pin "1") (pin "2") (instances (project "ChryslerScanner_V240_SD" (path "/b35850f9-3522-5e00-90df-092fcfbfe6bd/d24526bf-1665-5e09-804e-7766ac8ed522" (reference "R124") (unit 1)))))(wire (pts (xy 50.8 73.66) (xy 54.61 73.66)) (stroke (width 0) (type default)))(wire (pts (xy 62.23 73.66) (xy 66.04 73.66)) (stroke (width 0) (type default)))(wire (pts (xy 50.8 68.58) (xy 66.04 68.58)) (stroke (width 0) (type default)))(wire (pts (xy 66.04 68.58) (xy 66.04 73.66)) (stroke (width 0) (type default)))(global_label "N_R56_2"
+		(shape input)
+		(at 50.8 68.58 0)
+		(effects
+			(font
+				(size 0.95 0.95)
+			)
+			(justify left)
+		)
+		(property "Intersheetrefs" "${INTERSHEET_REFS}"
+			(at 50.8 68.58 0)
+			(hide yes)
+			(show_name no)
+			(do_not_autoplace no)
+			(effects
+				(font
+					(size 0.95 0.95)
+				)
+			)
+		)
+	)(text "VBB gate divider: 4.7k / 8.2k limits |Vgs| to 10.34V at the bounded 28V peak.\nAW9523 P0 must be configured push-pull; startup/default controls stay low." (at 25.4 153 0) (effects (font (size 1 1)) (justify left))))
