File: projects/chrysler-scanner/current/14_program-12.kicad_sch (KiCad schematic)
At the start: 9 parts, among them Q10 HSW4602, Q14 HSW4602

Commit message: Fix scanner protection, ADC isolation and health watchdog
Coordinate the bounded 12 V input clamp and programming FET/capacitor ratings, add powered-off ADC isolation, and supervise the AW9523B permit with a dedicated GPIO13 health heartbeat. Preserve original placements and document all deliberate source-PDF deviations.

Validation: native ERC and full DRC/parity/refill report zero findings; strict preservation/connectivity audit and final adversarial review pass within the documented prototype bounds. Regenerate Rev C PDF, BOM, manufacturing exports, processing sites and verified portable archives. Compatible firmware and bench/mechanical qualification remain required.
Parts:
- Q10: value HSW4602 -> DMC3071LVT-7
- Q14: value HSW4602 -> DMG6601LVT-7
- R70: value 4.7kΩ -> 4.7k 1%
- R71: value 1.1kΩ -> 8.2k 1%

Commit message: Finish Chrysler scanner CCD correction and procurement fabrication package
Parts:
- D17, D21: value MSK4005 -> PMEG4005; Assembly (none) -> PLACE; MPN (none) -> PMEG4005EGWX; Manufacturer (none) -> Nexperia; Procurement Source (none) -> https://assets.nexperia.com/documents/data-sheet/PMEG4005EG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
- Q10: Assembly (none) -> PLACE; MPN (none) -> DMC3071LVT-7; Manufacturer (none) -> Diodes Incorporated; Procurement Source (none) -> https://www.diodes.com/datasheet/download/DMC3071LVT.pdf
- Q14: Assembly (none) -> PLACE; MPN (none) -> DMG6601LVT-7; Manufacturer (none) -> Diodes Incorporated; Procurement Source (none) -> https://www.diodes.com/datasheet/download/DMG6601LVT.pdf
- R59, R69: Assembly (none) -> PLACE; MPN (none) -> CRCW060310K0FKEA; Manufacturer (none) -> Vishay; Procurement Source (none) -> https://www.vishay.com/docs/20035/dcrcwe3.pdf; Selected Power Rating (none) -> 0.1W; Tolerance (none) -> 1%
- R60, R70: Assembly (none) -> PLACE; MPN (none) -> CRCW06034K70FKEA; Manufacturer (none) -> Vishay; Procurement Source (none) -> https://www.vishay.com/docs/20035/dcrcwe3.pdf; Selected Power Rating (none) -> 0.1W; Tolerance (none) -> 1%
- R71: Assembly (none) -> PLACE; MPN (none) -> CRCW06038K20FKEA; Manufacturer (none) -> Vishay; Procurement Source (none) -> https://www.vishay.com/docs/20035/dcrcwe3.pdf; Selected Power Rating (none) -> 0.1W; Tolerance (none) -> 1%
Changed lines of the file:
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@@
 			)
 		)
-		(property "Datasheet" ""
+		(property "Datasheet" "https://www.diodes.com/datasheet/download/DMG6601LVT.pdf"
 			(at 168.402 73.66 0)
 			(hide yes)
@@
 			)
 		)
-	)
+(property "Manufacturer" "Diodes Incorporated" (at 0 0 0) (effects (font (size 1 1)) (hide yes)))
+(property "MPN" "DMG6601LVT-7" (at 0 0 0) (effects (font (size 1 1)) (hide yes)))
+(property "Procurement Source" "https://www.diodes.com/datasheet/download/DMG6601LVT.pdf" (at 0 0 0) (effects (font (size 1 1)) (hide yes)))
+(property "Assembly" "PLACE" (at 0 0 0) (effects (font (size 1 1)) (hide yes)))
+)
 	(symbol
 		(lib_id "ChryslerScanner:R59")
@@
 			)
 		)
-		(property "Datasheet" ""
+		(property "Datasheet" "https://www.vishay.com/docs/20035/dcrcwe3.pdf"
 			(at 33.02 101.6 0)
 			(hide yes)
@@
 			)
 		)
-	)
+(property "Manufacturer" "Vishay" (at 0 0 0) (effects (font (size 1 1)) (hide yes)))
+(property "MPN" "CRCW060310K0FKEA" (at 0 0 0) (effects (font (size 1 1)) (hide yes)))
+(property "Procurement Source" "https://www.vishay.com/docs/20035/dcrcwe3.pdf" (at 0 0 0) (effects (font (size 1 1)) (hide yes)))
+(property "Assembly" "PLACE" (at 0 0 0) (effects (font (size 1 1)) (hide yes)))
+(property "Tolerance" "1%" (at 0 0 0) (effects (font (size 1 1)) (hide yes)))
+(property "Selected Power Rating" "0.1W" (at 0 0 0) (effects (font (size 1 1)) (hide yes)))
+)
 	(symbol
 		(lib_id "ChryslerScanner:R60")
@@
 			)
 		)
-		(property "Datasheet" ""
+		(property "Datasheet" "https://www.vishay.com/docs/20035/dcrcwe3.pdf"
 			(at 50.8 60.96 0)
 			(hide yes)
@@
 			)
 		)
-	)
+(property "Manufacturer" "Vishay" (at 0 0 0) (effects (font (size 1 1)) (hide yes)))
+(property "MPN" "CRCW06034K70FKEA" (at 0 0 0) (effects (font (size 1 1)) (hide yes)))
+(property "Procurement Source" "https://www.vishay.com/docs/20035/dcrcwe3.pdf" (at 0 0 0) (effects (font (size 1 1)) (hide yes)))
+(property "Assembly" "PLACE" (at 0 0 0) (effects (font (size 1 1)) (hide yes)))
+(property "Tolerance" "1%" (at 0 0 0) (effects (font (size 1 1)) (hide yes)))
+(property "Selected Power Rating" "0.1W" (at 0 0 0) (effects (font (size 1 1)) (hide yes)))
+)
 	(symbol
 		(lib_id "ChryslerScanner:Q10")
@@
 			)
 		)
-		(property "Datasheet" ""
+		(property "Datasheet" "https://www.diodes.com/datasheet/download/DMC3071LVT.pdf"
 			(at 49.022 88.9 0)
 			(hide yes)
@@
 			)
 		)
-	)
+(property "Manufacturer" "Diodes Incorporated" (at 0 0 0) (effects (font (size 1 1)) (hide yes)))
+(property "MPN" "DMC3071LVT-7" (at 0 0 0) (effects (font (size 1 1)) (hide yes)))
+(property "Procurement Source" "https://www.diodes.com/datasheet/download/DMC3071LVT.pdf" (at 0 0 0) (effects (font (size 1 1)) (hide yes)))
+(property "Assembly" "PLACE" (at 0 0 0) (effects (font (size 1 1)) (hide yes)))
+)
 	(symbol
 		(lib_id "ChryslerScanner:R71")
@@
 			)
 		)
-		(property "Datasheet" ""
+		(property "Datasheet" "https://www.vishay.com/docs/20035/dcrcwe3.pdf"
 			(at 142.24 86.36 0)
 			(hide yes)
@@
 			)
 		)
-	)
+(property "Manufacturer" "Vishay" (at 0 0 0) (effects (font (size 1 1)) (hide yes)))
+(property "MPN" "CRCW06038K20FKEA" (at 0 0 0) (effects (font (size 1 1)) (hide yes)))
+(property "Procurement Source" "https://www.vishay.com/docs/20035/dcrcwe3.pdf" (at 0 0 0) (effects (font (size 1 1)) (hide yes)))
+(property "Assembly" "PLACE" (at 0 0 0) (effects (font (size 1 1)) (hide yes)))
+(property "Tolerance" "1%" (at 0 0 0) (effects (font (size 1 1)) (hide yes)))
+(property "Selected Power Rating" "0.1W" (at 0 0 0) (effects (font (size 1 1)) (hide yes)))
+)
 	(symbol
 		(lib_id "ChryslerScanner:R70")
@@
 			)
 		)
-		(property "Datasheet" ""
+		(property "Datasheet" "https://www.vishay.com/docs/20035/dcrcwe3.pdf"
 			(at 142.24 60.96 0)
 			(hide yes)
@@
 			)
 		)
-	)
+(property "Manufacturer" "Vishay" (at 0 0 0) (effects (font (size 1 1)) (hide yes)))
+(property "MPN" "CRCW06034K70FKEA" (at 0 0 0) (effects (font (size 1 1)) (hide yes)))
+(property "Procurement Source" "https://www.vishay.com/docs/20035/dcrcwe3.pdf" (at 0 0 0) (effects (font (size 1 1)) (hide yes)))
+(property "Assembly" "PLACE" (at 0 0 0) (effects (font (size 1 1)) (hide yes)))
+(property "Tolerance" "1%" (at 0 0 0) (effects (font (size 1 1)) (hide yes)))
+(property "Selected Power Rating" "0.1W" (at 0 0 0) (effects (font (size 1 1)) (hide yes)))
+)
 	(symbol
 		(lib_id "ChryslerScanner:Q10")
@@
 			)
 		)
-		(property "Datasheet" ""
+		(property "Datasheet" "https://www.diodes.com/datasheet/download/DMC3071LVT.pdf"
 			(at 76.962 73.66 0)
 			(hide yes)
@@
 			)
 		)
-	)
+(property "Manufacturer" "Diodes Incorporated" (at 0 0 0) (effects (font (size 1 1)) (hide yes)))
+(property "MPN" "DMC3071LVT-7" (at 0 0 0) (effects (font (size 1 1)) (hide yes)))
+(property "Procurement Source" "https://www.diodes.com/datasheet/download/DMC3071LVT.pdf" (at 0 0 0) (effects (font (size 1 1)) (hide yes)))
+(property "Assembly" "PLACE" (at 0 0 0) (effects (font (size 1 1)) (hide yes)))
+)
 	(symbol
 		(lib_id "power:GND")
@@
 			)
 		)
-		(property "Value" "MSK4005"
+		(property "Value" "PMEG4005"
 			(at 178.8274 92.39 0)
 			(show_name no)
@@
 			)
 		)
-		(property "Datasheet" ""
+		(property "Datasheet" "https://assets.nexperia.com/documents/data-sheet/PMEG4005EGW.pdf"
 			(at 170.18 91.44 0)
 			(hide yes)
@@
 			)
 		)
-	)
+(property "Manufacturer" "Nexperia" (at 0 0 0) (effects (font (size 1 1)) (hide yes)))
+(property "MPN" "PMEG4005EGWX" (at 0 0 0) (effects (font (size 1 1)) (hide yes)))
+(property "Procurement Source" "https://assets.nexperia.com/documents/data-sheet/PMEG4005EGW.pdf" (at 0 0 0) (effects (font (size 1 1)) (hide yes)))
+(property "Assembly" "PLACE" (at 0 0 0) (effects (font (size 1 1)) (hide yes)))
+)
 	(symbol
 		(lib_id "ChryslerScanner:D17")
@@
 			)
 		)
-		(property "Value" "MSK4005"
+		(property "Value" "PMEG4005"
 			(at 87.3874 92.39 0)
 			(show_name no)
@@
 			)
 		)
-		(property "Datasheet" ""
+		(property "Datasheet" "https://assets.nexperia.com/documents/data-sheet/PMEG4005EGW.pdf"
 			(at 78.74 91.44 0)
 			(hide yes)
@@
 			)
 		)
-	)
+(property "Manufacturer" "Nexperia" (at 0 0 0) (effects (font (size 1 1)) (hide yes)))
+(property "MPN" "PMEG4005EGWX" (at 0 0 0) (effects (font (size 1 1)) (hide yes)))
+(property "Procurement Source" "https://assets.nexperia.com/documents/data-sheet/PMEG4005EGW.pdf" (at 0 0 0) (effects (font (size 1 1)) (hide yes)))
+(property "Assembly" "PLACE" (at 0 0 0) (effects (font (size 1 1)) (hide yes)))
+)
 	(symbol
 		(lib_id "ChryslerScanner:R69")
@@
 			)
 		)
-		(property "Datasheet" ""
+		(property "Datasheet" "https://www.vishay.com/docs/20035/dcrcwe3.pdf"
 			(at 124.46 116.84 0)
 			(hide yes)
@@
 			)
 		)
-	)
+(property "Manufacturer" "Vishay" (at 0 0 0) (effects (font (size 1 1)) (hide yes)))
+(property "MPN" "CRCW060310K0FKEA" (at 0 0 0) (effects (font (size 1 1)) (hide yes)))
+(property "Procurement Source" "https://www.vishay.com/docs/20035/dcrcwe3.pdf" (at 0 0 0) (effects (font (size 1 1)) (hide yes)))
+(property "Assembly" "PLACE" (at 0 0 0) (effects (font (size 1 1)) (hide yes)))
+(property "Tolerance" "1%" (at 0 0 0) (effects (font (size 1 1)) (hide yes)))
+(property "Selected Power Rating" "0.1W" (at 0 0 0) (effects (font (size 1 1)) (hide yes)))
+)
 	(symbol
 		(lib_id "ChryslerScanner:Q14")
@@
 			)
 		)
-		(property "Datasheet" ""
+		(property "Datasheet" "https://www.diodes.com/datasheet/download/DMG6601LVT.pdf"
 			(at 140.462 104.14 0)
 			(hide yes)
@@
 			)
 		)
-	)
+(property "Manufacturer" "Diodes Incorporated" (at 0 0 0) (effects (font (size 1 1)) (hide yes)))
+(property "MPN" "DMG6601LVT-7" (at 0 0 0) (effects (font (size 1 1)) (hide yes)))
+(property "Procurement Source" "https://www.diodes.com/datasheet/download/DMG6601LVT.pdf" (at 0 0 0) (effects (font (size 1 1)) (hide yes)))
+(property "Assembly" "PLACE" (at 0 0 0) (effects (font (size 1 1)) (hide yes)))
+)
 	(symbol
 		(lib_id "power:GND")

Commit message: Refine programming drive, Eaton lands and mounting clearance
Parts:
- added R126: 8.2k 1%, footprints:R_0603_1608Metric, symbol ChryslerScanner:R126
- Q10: value DMC3071LVT-7 -> DMG6601LVT-7; MPN DMC3071LVT-7 -> DMG6601LVT-7; Procurement Source https://www.diodes.com/datasheet/download/DMC3071LVT.pdf -> https://www.diodes.com/datasheet/download/DMG6601LVT.pdf
Connections:
- net N_R60_2: now also R126.2; no longer Q10.6
- new net N_R126_1: Q10.6, R126.1
Other:
- note added: "VBB gate divider: 4.7k / 8.2k limits |Vgs| to 10.34V at the bounded 28V peak. AW9523 P0 must be configured push-pull; startup/default controls stay low."
Changed lines of the file:
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@@
-	(wire
-		(pts
-			(xy 50.8 73.66) (xy 66.04 73.66)
-		)
-		(stroke
-			(width 0)
-			(type default)
-		)
-	)
 	(wire
 		(pts
@@
 		(pts
 			(xy 78.74 48.26) (xy 78.74 63.5)
-		)
-		(stroke
-			(width 0)
-			(type default)
-		)
-	)
-	(wire
-		(pts
-			(xy 50.8 68.58) (xy 50.8 73.66)
 		)
 		(stroke
@@
 		)
 	)
-	(global_label "N_R60_2"
+	(global_label "N_R126_1"
 		(shape input)
 		(at 50.8 78.74 0)
@@
 			)
 		)
-		(property "Value" "DMC3071LVT-7"
+		(property "Value" "DMG6601LVT-7"
 			(at 60.7506 89.85 0)
 			(show_name no)
@@
 			)
 		)
-		(property "Datasheet" "https://www.diodes.com/datasheet/download/DMC3071LVT.pdf"
+		(property "Datasheet" "https://www.diodes.com/datasheet/download/DMG6601LVT.pdf"
 			(at 49.022 88.9 0)
 			(hide yes)
@@
 		)
 (property "Manufacturer" "Diodes Incorporated" (at 0 0 0) (effects (font (size 1 1)) (hide yes)))
-(property "MPN" "DMC3071LVT-7" (at 0 0 0) (effects (font (size 1 1)) (hide yes)))
-(property "Procurement Source" "https://www.diodes.com/datasheet/download/DMC3071LVT.pdf" (at 0 0 0) (effects (font (size 1 1)) (hide yes)))
+(property "MPN" "DMG6601LVT-7" (at 0 0 0) (effects (font (size 1 1)) (hide yes)))
+(property "Procurement Source" "https://www.diodes.com/datasheet/download/DMG6601LVT.pdf" (at 0 0 0) (effects (font (size 1 1)) (hide yes)))
 (property "Assembly" "PLACE" (at 0 0 0) (effects (font (size 1 1)) (hide yes)))
 )
@@
 			)
 		)
-		(property "Value" "DMC3071LVT-7"
+		(property "Value" "DMG6601LVT-7"
 			(at 88.6906 74.61 0)
 			(show_name no)
@@
 			)
 		)
-		(property "Datasheet" "https://www.diodes.com/datasheet/download/DMC3071LVT.pdf"
+		(property "Datasheet" "https://www.diodes.com/datasheet/download/DMG6601LVT.pdf"
 			(at 76.962 73.66 0)
 			(hide yes)
@@
 		)
 (property "Manufacturer" "Diodes Incorporated" (at 0 0 0) (effects (font (size 1 1)) (hide yes)))
-(property "MPN" "DMC3071LVT-7" (at 0 0 0) (effects (font (size 1 1)) (hide yes)))
-(property "Procurement Source" "https://www.diodes.com/datasheet/download/DMC3071LVT.pdf" (at 0 0 0) (effects (font (size 1 1)) (hide yes)))
+(property "MPN" "DMG6601LVT-7" (at 0 0 0) (effects (font (size 1 1)) (hide yes)))
+(property "Procurement Source" "https://www.diodes.com/datasheet/download/DMG6601LVT.pdf" (at 0 0 0) (effects (font (size 1 1)) (hide yes)))
 (property "Assembly" "PLACE" (at 0 0 0) (effects (font (size 1 1)) (hide yes)))
 )
@@
 		)
 	)
-)
+(symbol (lib_id "ChryslerScanner:R126") (at 58.42 73.66 0) (unit 1) (in_bom yes) (on_board yes) (dnp no)(property "Reference" "R126" (at 58.42 70.6 0) (effects (font (size 1 1))))(property "Value" "8.2k 1%" (at 58.42 76.7 0) (effects (font (size 1 1))))(property "Footprint" "footprints:R_0603_1608Metric" (at 58.42 73.66 0) (effects (font (size 1 1))(hide yes)))(property "Datasheet" "https://www.vishay.com/docs/20035/dcrcwe3.pdf" (at 58.42 73.66 0) (effects (font (size 1 1))(hide yes)))(property "Manufacturer" "Vishay" (at 58.42 73.66 0) (effects (font (size 1 1))(hide yes)))(property "MPN" "CRCW06038K20FKEA" (at 58.42 73.66 0) (effects (font (size 1 1))(hide yes)))(property "Procurement Source" "https://www.vishay.com/docs/20035/dcrcwe3.pdf" (at 58.42 73.66 0) (effects (font (size 1 1))(hide yes)))(property "Assembly" "PLACE" (at 58.42 73.66 0) (effects (font (size 1 1))(hide yes)))(property "Tolerance" "1%" (at 58.42 73.66 0) (effects (font (size 1 1))(hide yes)))(property "Selected Power Rating" "0.1W" (at 58.42 73.66 0) (effects (font (size 1 1))(hide yes)))(pin "1") (pin "2") (instances (project "ChryslerScanner_V240_SD" (path "/b35850f9-3522-5e00-90df-092fcfbfe6bd/66e1551e-d973-5aea-8598-c702df9afca6" (reference "R126") (unit 1)))))(wire (pts (xy 50.8 73.66) (xy 54.61 73.66)) (stroke (width 0) (type default)))(wire (pts (xy 62.23 73.66) (xy 66.04 73.66)) (stroke (width 0) (type default)))(wire (pts (xy 50.8 68.58) (xy 66.04 68.58)) (stroke (width 0) (type default)))(wire (pts (xy 66.04 68.58) (xy 66.04 73.66)) (stroke (width 0) (type default)))(global_label "N_R60_2"
+		(shape input)
+		(at 50.8 68.58 0)
+		(effects
+			(font
+				(size 0.95 0.95)
+			)
+			(justify left)
+		)
+		(property "Intersheetrefs" "${INTERSHEET_REFS}"
+			(at 50.8 68.58 0)
+			(hide yes)
+			(show_name no)
+			(do_not_autoplace no)
+			(effects
+				(font
+					(size 0.95 0.95)
+				)
+			)
+		)
+	)(text "VBB gate divider: 4.7k / 8.2k limits |Vgs| to 10.34V at the bounded 28V peak.\nAW9523 P0 must be configured push-pull; startup/default controls stay low." (at 25.4 153 0) (effects (font (size 1 1)) (justify left))))
